File: 1v25.kicad_sch (KiCad schematic)
At the start: 5 parts, among them U5 LMV321

Commit message: almost done with schematic
Parts:
- C14, C15: footprint (none) -> Capacitor_SMD:C_0402_1005Metric
- R5, R6: footprint (none) -> Resistor_SMD:R_0402_1005Metric
Changed lines of the file:
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@@
 (kicad_sch
-	(version 20260306)
+	(version 20260326)
 	(generator "eeschema")
-	(generator_version "10.0")
+	(generator_version "10.99")
 	(paper "A4")
 	(junction
-		(at 54.61 53.34)
+		(at 54.61 39.37)
 		(diameter 0)
 		(color 0 0 0 0)
@@
 	(wire
 		(pts
-			(xy 54.61 53.34) (xy 39.37 53.34)
+			(xy 54.61 39.37) (xy 55.88 39.37)
 		)
 		(stroke
@@
 	(wire
 		(pts
-			(xy 24.13 36.83) (xy 30.48 36.83)
+			(xy 54.61 53.34) (xy 39.37 53.34)
 		)
 		(stroke
@@
 	(wire
 		(pts
-			(xy 54.61 39.37) (xy 54.61 53.34)
+			(xy 24.13 36.83) (xy 30.48 36.83)
 		)
 		(stroke
@@
 	(wire
 		(pts
-			(xy 30.48 36.83) (xy 39.37 36.83)
+			(xy 54.61 39.37) (xy 54.61 53.34)
 		)
 		(stroke
@@
 	(wire
 		(pts
-			(xy 39.37 53.34) (xy 39.37 41.91)
+			(xy 30.48 36.83) (xy 39.37 36.83)
 		)
 		(stroke
@@
 	(wire
 		(pts
-			(xy 44.45 25.4) (xy 44.45 31.75)
+			(xy 39.37 53.34) (xy 39.37 41.91)
 		)
 		(stroke
@@
 		)
 	)
+	(wire
+		(pts
+			(xy 44.45 25.4) (xy 44.45 31.75)
+		)
+		(stroke
+			(width 0)
+			(type default)
+		)
+	)
 	(hierarchical_label "1V25"
 		(shape output)
-		(at 54.61 39.37 0)
+		(at 55.88 39.37 0)
 		(effects
 			(font
@@
 			)
 		)
-		(property "Footprint" ""
+		(property "Footprint" "Resistor_SMD:R_0402_1005Metric"
 			(at 28.702 40.64 90)
 			(hide yes)
@@
 			)
 		)
-		(property "Footprint" ""
+		(property "Footprint" "Resistor_SMD:R_0402_1005Metric"
 			(at 28.702 33.02 90)
 			(hide yes)
@@
 	)
 	(symbol
-		(lib_id "power:PWR_FLAG")
-		(at 54.61 53.34 270)
-		(unit 1)
-		(body_style 1)
-		(exclude_from_sim no)
-		(in_bom yes)
-		(on_board yes)
-		(in_pos_files yes)
-		(dnp no)
-		(fields_autoplaced yes)
-		(property "Reference" "#FLG04"
-			(at 56.515 53.34 0)
-			(hide yes)
-			(show_name no)
-			(do_not_autoplace no)
-			(effects
-				(font
-					(size 1.27 1.27)
-				)
-			)
-		)
-		(property "Value" "PWR_FLAG"
-			(at 58.42 53.3399 90)
-			(show_name no)
-			(do_not_autoplace no)
-			(effects
-				(font
-					(size 1.27 1.27)
-				)
-				(justify left)
-			)
-		)
-		(property "Footprint" ""
-			(at 54.61 53.34 0)
-			(hide yes)
-			(show_name no)
-			(do_not_autoplace no)
-			(effects
-				(font
-					(size 1.27 1.27)
-				)
-			)
-		)
-		(property "Datasheet" ""
-			(at 54.61 53.34 0)
-			(hide yes)
-			(show_name no)
-			(do_not_autoplace no)
-			(effects
-				(font
-					(size 1.27 1.27)
-				)
-			)
-		)
-		(property "Description" "Special symbol for telling ERC where power comes from"
-			(at 54.61 53.34 0)
-			(hide yes)
-			(show_name no)
-			(do_not_autoplace no)
-			(effects
-				(font
-					(size 1.27 1.27)
-				)
-			)
-		)
-		(pin "1"
-		)
-		(instances
-			(project "ht_better"
-				(path "/f8b7476c-07f9-4593-b1ba-2c61d2a9e349/116c6ec7-e28c-43c1-91b0-9b20e953211c"
-					(reference "#FLG04")
-					(unit 1)
-				)
-			)
-		)
-	)
-	(symbol
 		(lib_id "power:+5V")
 		(at 30.48 29.21 0)
@@
 			)
 		)
-		(property "Footprint" ""
+		(property "Footprint" "Capacitor_SMD:C_0402_1005Metric"
 			(at 25.0952 36.83 0)
 			(hide yes)
@@
 			)
 		)
-		(property "Footprint" ""
+		(property "Footprint" "Capacitor_SMD:C_0402_1005Metric"
 			(at 52.07 24.4348 0)
 			(hide yes)
