File: 25mhz_tcxo.kicad_sch (KiCad schematic)
At the start: 2 parts, among them U18 ECS-TXO-2520-33-250-AN-TR

Commit message: almost done with schematic
Parts:
- C138: footprint (none) -> Capacitor_SMD:C_0402_1005Metric
Changed lines of the file:
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@@
 (kicad_sch
-	(version 20260306)
+	(version 20260326)
 	(generator "eeschema")
-	(generator_version "10.0")
+	(generator_version "10.99")
 	(paper "A4")
 	(junction
@@
 			)
 		)
-		(property "Footprint" ""
+		(property "Footprint" "Capacitor_SMD:C_0402_1005Metric"
 			(at 80.01 23.1648 0)
 			(hide yes)
