File: buffer_2v5.kicad_sch (KiCad schematic)
At the start: 5 parts, among them U37 LMV321

Commit message: almost done with schematic
Changed lines of the file:
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@@
 (kicad_sch
-	(version 20260306)
+	(version 20260326)
 	(generator "eeschema")
-	(generator_version "10.0")
+	(generator_version "10.99")
 	(paper "A4")
 	(junction
@@
 	)
 	(junction
+		(at 57.15 36.83)
+		(diameter 0)
+		(color 0 0 0 0)
+	)
+	(junction
 		(at 46.99 29.21)
 		(diameter 0)
@@
 		(pts
 			(xy 57.15 36.83) (xy 57.15 50.8)
+		)
+		(stroke
+			(width 0)
+			(type default)
+		)
+	)
+	(wire
+		(pts
+			(xy 57.15 36.83) (xy 58.42 36.83)
 		)
 		(stroke
@@
 	(hierarchical_label "2V5"
 		(shape output)
-		(at 57.15 36.83 0)
+		(at 58.42 36.83 0)
 		(effects
 			(font
