File: mcu.kicad_sch (KiCad schematic)
At the start: 25 parts, among them J2 Conn_ARM_SWD_TagConnect_TC2030, U40 STM32H743VITx, X1 XL2EL89COI-111YLC-25M, X2 Q13FC1350000400

Commit message: almost done with schematic
Parts:
- added R121, R122: 2.2k, Resistor_SMD:R_0402_1005Metric, symbol Device:R
- C316, C317, C332: footprint (none) -> Capacitor_SMD:C_0603_1608Metric
- C318, C319, C320, C321, C322, C323, C324, C325, C326, C327, C328, C329, C330, C331: footprint (none) -> Capacitor_SMD:C_0402_1005Metric
- FB1: footprint (none) -> Inductor_SMD:L_0402_1005Metric
- R103, R104: footprint (none) -> Resistor_SMD:R_0402_1005Metric
- TP1: footprint (none) -> TestPoint:TestPoint_Pad_D1.5mm
Connections:
- net +3V3: now also R121.1, R122.1
- net SAI_MCLK: now reaches U40.1 (PE2)
- net CODEC_NRST: now reaches U40.15 (PC0)
- net CODEC_MOSI: now reaches U40.16 (PC1)
- net SAI_DIN: now reaches U40.2 (PE3)
- net VOL_POT: now reaches U40.23 (PA1)
- net RX_IN_2M: now reaches U40.24 (PA2)
- net RX_IN_70CM: now reaches U40.25 (PA3)
- net TX_DRIVER_BIAS: now reaches U40.28 (PA4)
- net TX_FINALS_BIAS: now reaches U40.29 (PA5)
- net SAI_WCLK: now reaches U40.3 (PE4)
- net RX_IF_MIXER1_2M_EN: now reaches U40.32 (PC4)
- net TX_LPF_SWITCH2: now reaches U40.33 (PC5)
- net FUNCTION_BTN: now reaches U40.34 (PB0)
- net PTT_BTN: now reaches U40.35 (PB1)
- net SQUELCH_BTN: now reaches U40.36 (PB2)
- net SAI_BCLK: now reaches U40.4 (PE5)
- net ROTARY_ENCODER_A: now reaches U40.41 (PE11)
- net ROTARY_ENCODER_BTN: now reaches U40.42 (PE12)
- net ROTARY_ENCODER_B: now reaches U40.43 (PE13)
- net DISPLAY_RESET: now reaches U40.46 (PB10)
- net DISPLAY_ENABLE: now reaches U40.47 (PB11)
- net SAI_DOUT: now reaches U40.5 (PE6)
- net DISPLAY_CS: now reaches U40.51 (PB12)
- net DISPLAY_SCK: now reaches U40.52 (PB13)
- net CODEC_MISO: now reaches U40.53 (PB14)
- net DISPLAY_SDA: now reaches U40.54 (PB15)
- net KEYPAD_ROW2: now reaches U40.55 (PD8)
- net KEYPAD_ROW3: now reaches U40.56 (PD9)
- net KEYPAD_ROW4: now reaches U40.57 (PD10)
- net KEYPAD_ROW5: now reaches U40.58 (PD11)
- net TX_BAND_SWITCH1: now reaches U40.59 (PD12)
- net TX_BAND_SWITCH2: now reaches U40.60 (PD13)
- net TX_MIXER_ENABLE: now reaches U40.61 (PD14)
- net TX_FDA_ENABLE: now reaches U40.62 (PD15)
- net TX_LPF_SWITCH1: now reaches U40.63 (PC6)
- net RX_IF_MIXER1_70CM_EN: now reaches U40.64 (PC7)
- net RX_IF_MIXER2_2M_PWDN: now reaches U40.65 (PC8)
- net RX_IF_MIXER2_70CM_PWDN: now reaches U40.66 (PC9)
- net PWR_SW: now reaches U40.7 (PC13)
- net RP2350_CS: now reaches U40.77 (PA15)
- net RP2350_SCK: now reaches U40.78 (PC10)
- net RP2350_MISO: now reaches U40.79 (PC11)
- net RP2350_MOSI: now reaches U40.80 (PC12)
- net CHARGER_INT: now reaches U40.81 (PD0)
- net CODEC_SCK: now reaches U40.84 (PD3)
- net KEYPAD_COL1: now reaches U40.85 (PD4)
- net KEYPAD_COL2: now reaches U40.86 (PD5)
- net KEYPAD_COL3: now reaches U40.87 (PD6)
- net KEYPAD_ROW1: now reaches U40.88 (PD7)
- net CODEC_CS: now reaches U40.90 (PB4)
- net TR_SWITCH: now reaches U40.91 (PB5)
- net I2C_SCL: now reaches U40.92 (PB6)
- net I2C_SCL: now also R121.2
- net I2C_SDA: now reaches U40.93 (PB7)
- net I2C_SDA: now also R122.2
- net DISPLAY_RS: now reaches U40.95 (PB8)
- net DISPLAY_PWM: now reaches U40.96 (PB9)
- no-connect marks 0 -> 18
