File: rf.kicad_sch (KiCad schematic)
At the start: 0 parts

Commit message: almost done with schematic
Other:
- sheet RX Frontend ports: added 1V25; removed 2V5
Changed lines of the file:
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@@
 (kicad_sch
-	(version 20260306)
+	(version 20260326)
 	(generator "eeschema")
-	(generator_version "10.0")
+	(generator_version "10.99")
 	(paper "A4")
 	(wire
@@
 	(wire
 		(pts
+			(xy 57.15 22.86) (xy 59.69 22.86)
+		)
+		(stroke
+			(width 0)
+			(type default)
+		)
+	)
+	(wire
+		(pts
 			(xy 34.29 100.33) (xy 35.56 100.33)
 		)
@@
 	(wire
 		(pts
-			(xy 88.9 31.75) (xy 90.17 31.75)
-		)
-		(stroke
-			(width 0)
-			(type default)
-		)
-	)
-	(wire
-		(pts
 			(xy 34.29 107.95) (xy 35.56 107.95)
 		)
@@
 		(pts
 			(xy 88.9 111.76) (xy 90.17 111.76)
+		)
+		(stroke
+			(width 0)
+			(type default)
+		)
+	)
+	(wire
+		(pts
+			(xy 88.9 24.13) (xy 90.17 24.13)
 		)
 		(stroke
@@
 		)
 	)
+	(hierarchical_label "1V25"
+		(shape input)
+		(at 88.9 24.13 180)
+		(effects
+			(font
+				(size 1.27 1.27)
+			)
+			(justify right)
+		)
+	)
 	(hierarchical_label "TX_FDA_DISABLE"
 		(shape input)
@@
 		)
 	)
-	(hierarchical_label "2V5"
-		(shape input)
-		(at 88.9 31.75 180)
-		(effects
-			(font
-				(size 1.27 1.27)
-			)
-			(justify right)
-		)
-	)
 	(hierarchical_label "RX_2M_LO_CE"
 		(shape input)
@@
 			)
 			(justify left)
+		)
+	)
+	(hierarchical_label "TR_SWITCH"
+		(shape input)
+		(at 57.15 22.86 270)
+		(effects
+			(font
+				(size 1.27 1.27)
+			)
+			(justify right)
 		)
 	)
@@
 			)
 		)
-		(pin "2V5" input
-			(at 90.17 31.75 180)
-			(effects
-				(font
-					(size 1.27 1.27)
-				)
-				(justify left)
-			)
-		)
 		(pin "70CM_IF1_MIXER_EN" input
 			(at 90.17 83.82 180)
@@
 			(effects
 				(font
+					(size 1.27 1.27)
+				)
+				(justify left)
+			)
+		)
+		(pin "1V25" input
+			(at 90.17 24.13 180)
+			(effects
+				(font
