File: tcxo_10.kicad_sch (KiCad schematic)
At the start: 2 parts, among them U13 ECS-TXO-2520MV-100-AY-TR

Commit message: almost done with schematic
Parts:
- C66: footprint (none) -> Capacitor_SMD:C_0402_1005Metric
Changed lines of the file:
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@@
 (kicad_sch
-	(version 20260306)
+	(version 20260326)
 	(generator "eeschema")
-	(generator_version "10.0")
+	(generator_version "10.99")
 	(paper "A4")
 	(junction
@@
 			)
 		)
-		(property "Footprint" ""
+		(property "Footprint" "Capacitor_SMD:C_0402_1005Metric"
 			(at 78.4352 36.83 0)
 			(hide yes)
