File: usb_c.kicad_sch (KiCad schematic)
At the start: 4 parts

Commit message: almost done with schematic
Parts:
- F1: footprint (none) -> Fuse:Fuse_1812_4532Metric
Connections:
- net USB_DN renamed USB_D-
- net USB_DP renamed USB_D+
Changed lines of the file:
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@@
 (kicad_sch
-	(version 20260306)
+	(version 20260326)
 	(generator "eeschema")
-	(generator_version "10.0")
+	(generator_version "10.99")
 	(paper "A4")
 	(junction
@@
 	)
 	(junction
+		(at 31.75 30.48)
+		(diameter 0)
+		(color 0 0 0 0)
+	)
+	(junction
 		(at 49.53 38.1)
 		(diameter 0)
@@
 	(wire
 		(pts
+			(xy 27.94 30.48) (xy 31.75 30.48)
+		)
+		(stroke
+			(width 0)
+			(type default)
+		)
+	)
+	(wire
+		(pts
 			(xy 52.07 53.34) (xy 44.45 53.34)
 		)
@@
 	(wire
 		(pts
+			(xy 31.75 30.48) (xy 31.75 31.75)
+		)
+		(stroke
+			(width 0)
+			(type default)
+		)
+	)
+	(wire
+		(pts
 			(xy 44.45 30.48) (xy 52.07 30.48)
 		)
@@
 	(wire
 		(pts
+			(xy 31.75 31.75) (xy 36.83 31.75)
+		)
+		(stroke
+			(width 0)
+			(type default)
+		)
+	)
+	(wire
+		(pts
 			(xy 35.56 40.64) (xy 40.64 40.64)
 		)
@@
 		)
 	)
-	(hierarchical_label "USB_DN"
+	(hierarchical_label "USB_D-"
 		(shape bidirectional)
 		(at 49.53 39.37 180)
@@
 		)
 	)
-	(hierarchical_label "USB_DP"
+	(hierarchical_label "USB_D+"
 		(shape bidirectional)
 		(at 46.99 43.18 180)
@@
 	)
 	(symbol
+		(lib_id "power:PWR_FLAG")
+		(at 31.75 30.48 0)
+		(unit 1)
+		(body_style 1)
+		(exclude_from_sim no)
+		(in_bom yes)
+		(on_board yes)
+		(in_pos_files yes)
+		(dnp no)
+		(fields_autoplaced yes)
+		(property "Reference" "#FLG09"
+			(at 31.75 28.575 0)
+			(hide yes)
+			(show_name no)
+			(do_not_autoplace no)
+			(effects
+				(font
+					(size 1.27 1.27)
+				)
+			)
+		)
+		(property "Value" "PWR_FLAG"
+			(at 31.75 25.4 0)
+			(show_name no)
+			(do_not_autoplace no)
+			(effects
+				(font
+					(size 1.27 1.27)
+				)
+			)
+		)
+		(property "Footprint" ""
+			(at 31.75 30.48 0)
+			(hide yes)
+			(show_name no)
+			(do_not_autoplace no)
+			(effects
+				(font
+					(size 1.27 1.27)
+				)
+			)
+		)
+		(property "Datasheet" ""
+			(at 31.75 30.48 0)
+			(hide yes)
+			(show_name no)
+			(do_not_autoplace no)
+			(effects
+				(font
+					(size 1.27 1.27)
+				)
+			)
+		)
+		(property "Description" "Special symbol for telling ERC where power comes from"
+			(at 31.75 30.48 0)
+			(hide yes)
+			(show_name no)
+			(do_not_autoplace no)
+			(effects
+				(font
+					(size 1.27 1.27)
+				)
+			)
+		)
+		(pin "1"
+		)
+		(instances
+			(project "ht_better"
+				(path "/f8b7476c-07f9-4593-b1ba-2c61d2a9e349/fbdb0304-33c0-4b24-99e5-6b0dd4dc94e1"
+					(reference "#FLG09")
+					(unit 1)
+				)
+			)
+		)
+	)
+	(symbol
 		(lib_id "power:GND")
 		(at 35.56 45.72 0)
@@
 	(symbol
 		(lib_id "power:VBUS")
-		(at 36.83 31.75 90)
+		(at 27.94 30.48 90)
 		(unit 1)
 		(body_style 1)
@@
 		(fields_autoplaced yes)
 		(property "Reference" "#PWR0439"
-			(at 40.64 31.75 0)
+			(at 31.75 30.48 0)
 			(hide yes)
 			(show_name no)
@@
 		)
 		(property "Value" "VBUS"
-			(at 33.02 31.7499 90)
+			(at 24.13 30.4799 90)
 			(show_name no)
 			(do_not_autoplace no)
@@
 		)
 		(property "Footprint" ""
-			(at 36.83 31.75 0)
+			(at 27.94 30.48 0)
 			(hide yes)
 			(show_name no)
@@
 		)
 		(property "Datasheet" ""
-			(at 36.83 31.75 0)
+			(at 27.94 30.48 0)
 			(hide yes)
 			(show_name no)
@@
 		)
 		(property "Description" "Power symbol creates a global label with name \"VBUS\""
-			(at 36.83 31.75 0)
+			(at 27.94 30.48 0)
 			(hide yes)
 			(show_name no)
@@
 			)
 		)
-		(property "Footprint" ""
+		(property "Footprint" "Fuse:Fuse_1812_4532Metric"
 			(at 45.72 30.48 0)
 			(hide yes)
