File: 2m_lna.kicad_sch (KiCad schematic)
At the start: 6 parts, among them U10 PGA-103+

Commit message: almost done with schematic
Parts:
- C33, C34, C35, C36: footprint (none) -> Capacitor_SMD:C_0402_1005Metric
Changed lines of the file:
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@@
 (kicad_sch
-	(version 20260306)
+	(version 20260326)
 	(generator "eeschema")
-	(generator_version "10.0")
+	(generator_version "10.99")
 	(paper "A4")
 	(junction
@@
 			)
 		)
-		(property "Footprint" ""
+		(property "Footprint" "Capacitor_SMD:C_0402_1005Metric"
 			(at 35.56 24.4348 0)
 			(hide yes)
@@
 			)
 		)
-		(property "Footprint" ""
+		(property "Footprint" "Capacitor_SMD:C_0402_1005Metric"
 			(at 35.56 31.4452 0)
 			(hide yes)
@@
 			)
 		)
-		(property "Footprint" ""
+		(property "Footprint" "Capacitor_SMD:C_0402_1005Metric"
 			(at 58.42 53.0352 0)
 			(hide yes)
@@
 			)
 		)
-		(property "Footprint" ""
+		(property "Footprint" "Capacitor_SMD:C_0402_1005Metric"
 			(at 58.42 41.6052 0)
 			(hide yes)

Commit message: almost done assigning footprints
Parts:
- L16: footprint (none) -> Inductor_SMD:L_0603_1608Metric
Changed lines of the file:
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@@
 			)
 		)
-		(property "Footprint" ""
+		(property "Footprint" "Inductor_SMD:L_0603_1608Metric"
 			(at 44.45 36.83 0)
 			(hide yes)
