File: 3v3.kicad_sch (KiCad schematic)
At the start: 7 parts, among them U2 TPS564208DDCR

Commit message: almost done with schematic
Parts:
- C4: footprint (none) -> Capacitor_SMD:C_0603_1608Metric
- C5: footprint (none) -> Capacitor_SMD:C_0402_1005Metric
- C6: footprint (none) -> Capacitor_SMD:C_0805_2012Metric
- R1, R2: footprint (none) -> Resistor_SMD:R_0402_1005Metric
Changed lines of the file:
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@@
 (kicad_sch
-	(version 20260306)
+	(version 20260326)
 	(generator "eeschema")
-	(generator_version "10.0")
+	(generator_version "10.99")
 	(paper "A4")
 	(junction
@@
 			)
 		)
-		(property "Footprint" ""
+		(property "Footprint" "Capacitor_SMD:C_0805_2012Metric"
 			(at 84.7852 38.1 0)
 			(hide yes)
@@
 			)
 		)
-		(property "Footprint" ""
+		(property "Footprint" "Capacitor_SMD:C_0402_1005Metric"
 			(at 58.42 21.8948 0)
 			(hide yes)
@@
 			)
 		)
-		(property "Footprint" ""
+		(property "Footprint" "Capacitor_SMD:C_0603_1608Metric"
 			(at 31.4452 44.45 0)
 			(hide yes)
@@
 			)
 		)
-		(property "Footprint" ""
+		(property "Footprint" "Resistor_SMD:R_0402_1005Metric"
 			(at 70.612 41.91 90)
 			(hide yes)
@@
 			)
 		)
-		(property "Footprint" ""
+		(property "Footprint" "Resistor_SMD:R_0402_1005Metric"
 			(at 70.612 34.29 90)
 			(hide yes)

Commit message: almost done assigning footprints
Parts:
- L1: footprint (none) -> Inductor_SMD:L_1008_2520Metric
Changed lines of the file:
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@@
 			)
 		)
-		(property "Footprint" ""
+		(property "Footprint" "Inductor_SMD:L_1008_2520Metric"
 			(at 60.96 30.48 0)
 			(hide yes)
