File: battery_charger.kicad_sch (KiCad schematic)
At the start: 21 parts, among them U38 BQ25798

Commit message: almost done with schematic
Parts:
- added C381, C382, C383: 10uF, Capacitor_SMD:C_0603_1608Metric, symbol Device:C
- added C384: 100nF, Capacitor_SMD:C_0402_1005Metric, symbol Device:C
- C301, C302, C304, C306: footprint (none) -> Capacitor_SMD:C_0402_1005Metric
- C303, C305, C307, C308, C309, C310, C311, C312: footprint (none) -> Capacitor_SMD:C_0603_1608Metric
- R100, R95, R96, R97, R98, R99, TH1: footprint (none) -> Resistor_SMD:R_0402_1005Metric
Connections:
- net GND: now also C381.2, C382.2, C383.2, C384.2
- net at U38.29 (PMID): now also C381.1, C382.1, C383.1, C384.1

Commit message: almost done assigning footprints
Parts:
- L99: footprint (none) -> Inductor_SMD:L_1008_2520Metric
Changed lines of the file:
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@@
 			)
 		)
-		(property "Footprint" ""
+		(property "Footprint" "Inductor_SMD:L_1008_2520Metric"
 			(at 90.17 38.1 0)
 			(hide yes)
