File: codec.kicad_sch (KiCad schematic)
At the start: 15 parts, among them U41 TLV320AIC3254IRHBT

Commit message: almost done with schematic
Parts:
- C343, C344, C349: footprint (none) -> Capacitor_SMD:C_0402_1005Metric
- C345, C346, C347, C348, C350, C351, C352: footprint (none) -> Capacitor_SMD:C_0603_1608Metric
- R115, R116, R117: footprint (none) -> Resistor_SMD:R_0402_1005Metric
Changed lines of the file:
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@@
 (kicad_sch
-	(version 20260306)
+	(version 20260326)
 	(generator "eeschema")
-	(generator_version "10.0")
+	(generator_version "10.99")
 	(paper "A4")
 	(junction
@@
 			)
 		)
-		(property "Footprint" ""
+		(property "Footprint" "Capacitor_SMD:C_0402_1005Metric"
 			(at 37.7952 86.36 0)
 			(hide yes)
@@
 			)
 		)
-		(property "Footprint" ""
+		(property "Footprint" "Capacitor_SMD:C_0402_1005Metric"
 			(at 114.6048 63.5 0)
 			(hide yes)
@@
 			)
 		)
-		(property "Footprint" ""
+		(property "Footprint" "Capacitor_SMD:C_0603_1608Metric"
 			(at 26.9748 71.12 0)
 			(hide yes)
@@
 			)
 		)
-		(property "Footprint" ""
+		(property "Footprint" "Capacitor_SMD:C_0603_1608Metric"
 			(at 99.06 23.1648 0)
 			(hide yes)
@@
 			)
 		)
-		(property "Footprint" ""
+		(property "Footprint" "Capacitor_SMD:C_0603_1608Metric"
 			(at 107.95 31.4452 0)
 			(hide yes)
@@
 			)
 		)
-		(property "Footprint" ""
+		(property "Footprint" "Resistor_SMD:R_0402_1005Metric"
 			(at 120.65 25.908 90)
 			(hide yes)
@@
 			)
 		)
-		(property "Footprint" ""
+		(property "Footprint" "Capacitor_SMD:C_0603_1608Metric"
 			(at 21.8948 86.36 0)
 			(hide yes)
@@
 			)
 		)
-		(property "Footprint" ""
+		(property "Footprint" "Capacitor_SMD:C_0402_1005Metric"
 			(at 26.9748 78.74 0)
 			(hide yes)
@@
 			)
 		)
-		(property "Footprint" ""
+		(property "Footprint" "Capacitor_SMD:C_0603_1608Metric"
 			(at 29.21 106.9848 0)
 			(hide yes)
@@
 			)
 		)
-		(property "Footprint" ""
+		(property "Footprint" "Resistor_SMD:R_0402_1005Metric"
 			(at 115.062 38.1 90)
 			(hide yes)
@@
 			)
 		)
-		(property "Footprint" ""
+		(property "Footprint" "Resistor_SMD:R_0402_1005Metric"
 			(at 31.242 57.15 90)
 			(hide yes)
@@
 			)
 		)
-		(property "Footprint" ""
+		(property "Footprint" "Capacitor_SMD:C_0603_1608Metric"
 			(at 103.1748 63.5 0)
 			(hide yes)
@@
 			)
 		)
-		(property "Footprint" ""
+		(property "Footprint" "Capacitor_SMD:C_0603_1608Metric"
 			(at 29.21 95.5548 0)
 			(hide yes)

Commit message: almost done assigning footprints
Parts:
- removed MK1: Microphone_Condenser, symbol Device:Microphone_Condenser
- added MIC1: B4013AM423-092, easyeda2kicad:MIC-SMD_BD4.0_B4013AM423-093-1, symbol easyeda2kicad:B4013AM423-092
Connections:
- net at C351.2, R117.1: now also MIC1.1 (+)
- net at C352.2, R116.1: now also MIC1.2 (-)
Changed lines of the file:
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@@
 	(paper "A4")
+	(junction
+		(at 116.84 34.29)
+		(diameter 0)
+		(color 0 0 0 0)
+	)
 	(junction
 		(at 91.44 76.2)
@@
 	)
 	(junction
-		(at 116.84 34.29)
-		(diameter 0)
-		(color 0 0 0 0)
-	)
-	(junction
 		(at 27.94 71.12)
-		(diameter 0)
-		(color 0 0 0 0)
-	)
-	(junction
-		(at 116.84 24.13)
 		(diameter 0)
 		(color 0 0 0 0)
@@
 	)
 	(junction
+		(at 115.57 24.13)
+		(diameter 0)
+		(color 0 0 0 0)
+	)
+	(junction
 		(at 26.67 71.12)
 		(diameter 0)
@@
 	(wire
 		(pts
-			(xy 99.06 24.13) (xy 116.84 24.13)
+			(xy 99.06 24.13) (xy 115.57 24.13)
 		)
 		(stroke
@@
 	(wire
 		(pts
+			(xy 115.57 24.13) (xy 116.84 24.13)
+		)
+		(stroke
+			(width 0)
+			(type default)
+		)
+	)
+	(wire
+		(pts
 			(xy 31.75 107.95) (xy 31.75 76.2)
 		)
@@
 	(wire
 		(pts
+			(xy 115.57 27.94) (xy 115.57 24.13)
+		)
+		(stroke
+			(width 0)
+			(type default)
+		)
+	)
+	(wire
+		(pts
 			(xy 26.67 72.39) (xy 26.67 71.12)
 		)
@@
 	(wire
 		(pts
+			(xy 116.84 34.29) (xy 116.84 33.02)
+		)
+		(stroke
+			(width 0)
+			(type default)
+		)
+	)
+	(wire
+		(pts
 			(xy 33.02 60.96) (xy 50.8 60.96)
 		)
@@
 	(wire
 		(pts
+			(xy 129.54 27.94) (xy 115.57 27.94)
+		)
+		(stroke
+			(width 0)
+			(type default)
+		)
+	)
+	(wire
+		(pts
 			(xy 27.94 71.12) (xy 50.8 71.12)
 		)
@@
 		(pts
 			(xy 104.14 63.5) (xy 115.57 63.5)
+		)
+		(stroke
+			(width 0)
+			(type default)
+		)
+	)
+	(wire
+		(pts
+			(xy 116.84 33.02) (xy 129.54 33.02)
 		)
 		(stroke
@@
 	)
 	(symbol
-		(lib_id "Device:Microphone_Condenser")
-		(at 116.84 29.21 0)
-		(unit 1)
-		(body_style 1)
-		(exclude_from_sim no)
-		(in_bom yes)
-		(on_board yes)
-		(in_pos_files yes)
-		(dnp no)
-		(fields_autoplaced yes)
-		(property "Reference" "MK1"
-			(at 120.65 27.2414 0)
-			(show_name no)
-			(do_not_autoplace no)
-			(effects
-				(font
-					(size 1.27 1.27)
-				)
-				(justify left)
-			)
-		)
-		(property "Value" "Microphone_Condenser"
-			(at 120.65 29.7814 0)
-			(show_name no)
-			(do_not_autoplace no)
-			(effects
-				(font
-					(size 1.27 1.27)
-				)
-				(justify left)
-			)
-		)
-		(property "Footprint" ""
-			(at 116.84 26.67 90)
-			(hide yes)
-			(show_name no)
-			(do_not_autoplace no)
-			(effects
-				(font
-					(size 1.27 1.27)
-				)
-			)
-		)
-		(property "Datasheet" ""
-			(at 116.84 26.67 90)
-			(hide yes)
-			(show_name no)
-			(do_not_autoplace no)
-			(effects
-				(font
-					(size 1.27 1.27)
-				)
-			)
-		)
-		(property "Description" "Condenser microphone"
-			(at 116.84 29.21 0)
-			(hide yes)
-			(show_name no)
-			(do_not_autoplace no)
-			(effects
-				(font
-					(size 1.27 1.27)
-				)
-			)
-		)
-		(pin "1"
-		)
-		(pin "2"
-		)
-		(instances
-			(project "ht_better"
-				(path "/f8b7476c-07f9-4593-b1ba-2c61d2a9e349/7d41882d-0176-419a-87e2-f78eee2f944c/34a9ad3c-055c-4b99-a1d1-7126d401cb12"
-					(reference "MK1")
-					(unit 1)
-				)
-			)
-		)
-	)
-	(symbol
 		(lib_id "Device:C")
 		(at 104.14 67.31 180)
@@
 					(unit 1)
 				)
+			)
+		)
+	)
+	(symbol
+		(lib_id "easyeda2kicad:B4013AM423-092")
+		(at 134.62 30.48 270)
+		(unit 1)
+		(body_style 1)
+		(exclude_from_sim no)
+		(in_bom yes)
+		(on_board yes)
+		(in_pos_files yes)
+		(dnp no)
+		(fields_autoplaced yes)
+		(property "Reference" "MIC1"
+			(at 143.51 29.2099 90)
+			(show_name no)
+			(do_not_autoplace no)
+			(effects
+				(font
+					(size 1.27 1.27)
+				)
+				(justify left)
+			)
+		)
+		(property "Value" "B4013AM423-092"
+			(at 143.51 31.7499 90)
+			(show_name no)
+			(do_not_autoplace no)
+			(effects
+				(font
+					(size 1.27 1.27)
+				)
+				(justify left)
+			)
+		)
+		(property "Footprint" "easyeda2kicad:MIC-SMD_BD4.0_B4013AM423-093-1"
+			(at 121.92 30.48 0)
+			(hide yes)
+			(show_name no)
+			(do_not_autoplace no)
+			(effects
+				(font
+					(size 1.27 1.27)
+				)
+			)
+		)
+		(property "Datasheet" ""
+			(at 134.62 30.48 0)
+			(hide yes)
+			(show_name no)
+			(do_not_autoplace no)
+			(effects
+				(font
+					(size 1.27 1.27)
+				)
+			)
+		)
+		(property "Description" ""
+			(at 134.62 30.48 0)
+			(hide yes)
+			(show_name no)
+			(do_not_autoplace no)
+			(effects
+				(font
+					(size 1.27 1.27)
+				)
+			)
+		)
+		(property "LCSC Part" "C5160218"
+			(at 119.38 30.48 0)
+			(hide yes)
+			(show_name no)
+			(do_not_autoplace no)
+			(effects
+				(font
+					(size 1.27 1.27)
+				)
+			)
+		)
+		(pin "1"
+		)
+		(pin "2"
+		)
+		(instances
+			(project "ht_better"
+				(path "/f8b7476c-07f9-4593-b1ba-2c61d2a9e349/7d41882d-0176-419a-87e2-f78eee2f944c/34a9ad3c-055c-4b99-a1d1-7126d401cb12"
+					(reference "MIC1")
+					(unit 1)
+				)
