File: in_safety.kicad_sch (KiCad schematic)
At the start: 3 parts

Commit message: almost done with schematic
Parts:
- C16: footprint (none) -> Capacitor_SMD:C_0402_1005Metric
- R7: footprint (none) -> Resistor_SMD:R_0603_1608Metric
Changed lines of the file:
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@@
 (kicad_sch
-	(version 20260306)
+	(version 20260326)
 	(generator "eeschema")
-	(generator_version "10.0")
+	(generator_version "10.99")
 	(paper "A4")
 	(junction
@@
 			)
 		)
-		(property "Footprint" ""
+		(property "Footprint" "Capacitor_SMD:C_0402_1005Metric"
 			(at 64.77 30.7848 0)
 			(hide yes)
@@
 			)
 		)
-		(property "Footprint" ""
+		(property "Footprint" "Resistor_SMD:R_0603_1608Metric"
 			(at 45.212 27.94 90)
 			(hide yes)

Commit message: almost done assigning footprints
Parts:
- GD1: footprint (none) -> Fuse:Fuse_1206_3216Metric
Changed lines of the file:
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@@
 			)
 		)
-		(property "Footprint" ""
+		(property "Footprint" "Fuse:Fuse_1206_3216Metric"
 			(at 29.21 26.67 90)
 			(hide yes)
