File: volume_power_pot.kicad_sch (KiCad schematic)
At the start: 3 parts

Commit message: almost done with schematic
Parts:
- C339, C340: footprint (none) -> Capacitor_SMD:C_0402_1005Metric
- R112: footprint (none) -> Resistor_SMD:R_0402_1005Metric
Changed lines of the file:
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@@
 (kicad_sch
-	(version 20260306)
+	(version 20260326)
 	(generator "eeschema")
-	(generator_version "10.0")
+	(generator_version "10.99")
 	(paper "A4")
 	(junction
@@
 			)
 		)
-		(property "Footprint" ""
+		(property "Footprint" "Capacitor_SMD:C_0402_1005Metric"
 			(at 44.1452 35.56 0)
 			(hide yes)
@@
 			)
 		)
-		(property "Footprint" ""
+		(property "Footprint" "Resistor_SMD:R_0402_1005Metric"
 			(at 52.832 31.75 90)
 			(hide yes)
@@
 			)
 		)
-		(property "Footprint" ""
+		(property "Footprint" "Capacitor_SMD:C_0402_1005Metric"
 			(at 67.0052 27.94 0)
 			(hide yes)

Commit message: finish schematic
Changed lines of the file:
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@@
 		(body_style 1)
 		(exclude_from_sim no)
-		(in_bom no)
-		(on_board no)
+		(in_bom yes)
+		(on_board yes)
 		(in_pos_files yes)
 		(dnp no)
@@
 			)
 		)
-		(property "Value" ""
+		(property "Value" "RK09711110EL"
 			(at 35.56 26.67 0)
 			(show_name no)
@@
 			)
 		)
-		(property "Footprint" ""
+		(property "Footprint" "footprints:RK09711110EL"
 			(at 35.56 26.67 0)
 			(hide yes)
