File: ht_better.kicad_pcb (KiCad board)
At the start: 2 copper layers, 0 parts

Commit message: almost done assigning footprints
Parts:
- added C1: 100nF, Capacitor_SMD:C_0402_1005Metric, F.Cu at (293.6, 82.0)
- added C10: 100nF, Capacitor_SMD:C_0402_1005Metric, F.Cu at (288.3, 138.5)
- added C100: 68pF, Capacitor_SMD:C_0402_1005Metric, F.Cu at (233.3, 91.9)
- added C101: 68pF, Capacitor_SMD:C_0402_1005Metric, F.Cu at (236.2, 82.0)
- added C102: 470pF, Capacitor_SMD:C_0402_1005Metric, F.Cu at (236.2, 84.0)
- added C103: 1nF, Capacitor_SMD:C_0402_1005Metric, F.Cu at (236.2, 86.0)
- added C104: 1uF, Capacitor_SMD:C_0603_1608Metric, F.Cu at (227.0, 82.3)
- added C105: 1nF, Capacitor_SMD:C_0402_1005Metric, F.Cu at (194.0, 141.1)
- added C106: 12pF, Capacitor_SMD:C_0402_1005Metric, F.Cu at (194.0, 143.1)
- added C107: 12pF, Capacitor_SMD:C_0402_1005Metric, F.Cu at (194.0, 145.1)
- added C108: 1nF, Capacitor_SMD:C_0402_1005Metric, F.Cu at (238.3, 150.4)
- added C109: 1nF, Capacitor_SMD:C_0402_1005Metric, F.Cu at (238.3, 152.4)
- added C11: 1uF, Capacitor_SMD:C_0603_1608Metric, F.Cu at (234.8, 166.6)
- added C110: 1nF, Capacitor_SMD:C_0402_1005Metric, F.Cu at (238.3, 154.4)
- added C111: 100nF, Capacitor_SMD:C_0402_1005Metric, F.Cu at (241.2, 150.4)
- added C112: 100nF, Capacitor_SMD:C_0402_1005Metric, F.Cu at (241.2, 152.4)
- added C113: 1nF, Capacitor_SMD:C_0402_1005Metric, F.Cu at (241.2, 154.4)
- added C114: 100nF, Capacitor_SMD:C_0402_1005Metric, F.Cu at (244.0, 150.4)
- added C115: 1nF, Capacitor_SMD:C_0402_1005Metric, F.Cu at (244.0, 152.4)
- added C116: 1nF, Capacitor_SMD:C_0402_1005Metric, F.Cu at (244.0, 154.4)
- added C117: 470nF, Capacitor_SMD:C_0603_1608Metric, F.Cu at (234.8, 150.7)
- added C118: 470nF, Capacitor_SMD:C_0603_1608Metric, F.Cu at (234.8, 153.2)
- added C119: 1uF, Capacitor_SMD:C_0603_1608Metric, F.Cu at (234.8, 155.7)
- added C12: 2.2uF, Capacitor_SMD:C_0603_1608Metric, F.Cu at (234.8, 169.1)
- added C120: 1uF, Capacitor_SMD:C_0603_1608Metric, F.Cu at (234.8, 158.2)
- added C121: 39pF, Capacitor_SMD:C_0402_1005Metric, F.Cu at (254.2, 144.2)
- added C122: 1.1pF, Capacitor_SMD:C_0402_1005Metric, F.Cu at (254.2, 146.2)
- added C123: 68pF, Capacitor_SMD:C_0402_1005Metric, F.Cu at (254.2, 148.2)
- added C124: 1.1pF, Capacitor_SMD:C_0402_1005Metric, F.Cu at (254.2, 150.2)
- added C125: 39pF, Capacitor_SMD:C_0402_1005Metric, F.Cu at (254.2, 152.1)
- added C126: 470pF, Capacitor_SMD:C_0402_1005Metric, F.Cu at (281.2, 144.2)
- added C127: 470pF, Capacitor_SMD:C_0402_1005Metric, F.Cu at (281.2, 146.1)
- added C128: 100pF, Capacitor_SMD:C_0402_1005Metric, F.Cu at (281.2, 148.1)
- added C129: 100nF, Capacitor_SMD:C_0402_1005Metric, F.Cu at (281.2, 150.1)
- added C13: 2.2uF, Capacitor_SMD:C_0603_1608Metric, F.Cu at (234.8, 171.6)
- added C130: 36pF, Capacitor_SMD:C_0402_1005Metric, F.Cu at (254.2, 164.2)
- added C131: 1.3pF, Capacitor_SMD:C_0402_1005Metric, F.Cu at (254.2, 166.1)
- added C132: 36pF, Capacitor_SMD:C_0402_1005Metric, F.Cu at (254.2, 168.1)
- added C133: 100nF, Capacitor_SMD:C_0402_1005Metric, F.Cu at (269.4, 132.3)
- added C134: 100nF, Capacitor_SMD:C_0402_1005Metric, F.Cu at (269.4, 134.3)
- added C135: 100nF, Capacitor_SMD:C_0402_1005Metric, F.Cu at (269.4, 136.2)
- added C136: 100nF, Capacitor_SMD:C_0402_1005Metric, F.Cu at (269.4, 138.2)
- added C137: 100nF, Capacitor_SMD:C_0402_1005Metric, F.Cu at (269.4, 140.2)
- added C138: 100nF, Capacitor_SMD:C_0402_1005Metric, F.Cu at (292.5, 148.6)
- added C139: 62pF, Capacitor_SMD:C_0402_1005Metric, F.Cu at (197.5, 154.9)
- added C14: 100nF, Capacitor_SMD:C_0402_1005Metric, F.Cu at (259.1, 160.3)
- added C140: 100pF, Capacitor_SMD:C_0402_1005Metric, F.Cu at (197.5, 156.9)
- added C141: 62pF, Capacitor_SMD:C_0402_1005Metric, F.Cu at (197.5, 158.9)
- added C142: 62pF, Capacitor_SMD:C_0402_1005Metric, F.Cu at (197.5, 162.8)
- added C143: 100pF, Capacitor_SMD:C_0402_1005Metric, F.Cu at (197.5, 164.8)
- added C144: 62pF, Capacitor_SMD:C_0402_1005Metric, F.Cu at (197.5, 166.8)
- added C145: 100nF, Capacitor_SMD:C_0402_1005Metric, F.Cu at (271.5, 82.0)
- added C146: 4.7pF, Capacitor_SMD:C_0402_1005Metric, F.Cu at (271.5, 84.0)
- added C147: 4.7pF, Capacitor_SMD:C_0402_1005Metric, F.Cu at (271.5, 86.0)
- added C148: 1uF, Capacitor_SMD:C_0603_1608Metric, F.Cu at (262.2, 82.3)
- added C149: 1uF, Capacitor_SMD:C_0603_1608Metric, F.Cu at (262.2, 84.8)
- added C15: 100nF, Capacitor_SMD:C_0402_1005Metric, F.Cu at (259.1, 162.3)
- added C150: 1uF, Capacitor_SMD:C_0603_1608Metric, F.Cu at (262.2, 87.3)
- added C151: 1uF, Capacitor_SMD:C_0603_1608Metric, F.Cu at (262.2, 89.8)
- added C152: 1uF, Capacitor_SMD:C_0603_1608Metric, F.Cu at (262.2, 92.4)
- added C153: 1uF, Capacitor_SMD:C_0603_1608Metric, F.Cu at (262.2, 94.9)
- added C154: 10pF, Capacitor_SMD:C_0402_1005Metric, F.Cu at (279.3, 82.0)
- added C155: 4.7pF, Capacitor_SMD:C_0402_1005Metric, F.Cu at (279.3, 84.0)
- added C156: 100nF, Capacitor_SMD:C_0402_1005Metric, F.Cu at (279.3, 86.0)
- added C157: 1uF, Capacitor_SMD:C_0603_1608Metric, F.Cu at (282.7, 90.7)
- added C158: 100nF, Capacitor_SMD:C_0402_1005Metric, F.Cu at (279.3, 88.0)
- added C159: 100nF, Capacitor_SMD:C_0402_1005Metric, F.Cu at (279.3, 89.9)
- added C16: 470pF, Capacitor_SMD:C_0402_1005Metric, F.Cu at (285.8, 114.0)
- added C160: 10pF, Capacitor_SMD:C_0402_1005Metric, F.Cu at (279.3, 91.9)
- added C161: 4.7pF, Capacitor_SMD:C_0402_1005Metric, F.Cu at (279.3, 93.9)
- added C162: 100nF, Capacitor_SMD:C_0402_1005Metric, F.Cu at (279.3, 95.8)
- added C163: 1uF, Capacitor_SMD:C_0603_1608Metric, F.Cu at (282.7, 93.2)
- added C164: 1uF, Capacitor_SMD:C_0603_1608Metric, F.Cu at (181.5, 144.3)
- added C165: 1uF, Capacitor_SMD:C_0603_1608Metric, F.Cu at (181.5, 146.8)
- added C166: 470pF, Capacitor_SMD:C_0402_1005Metric_Pad0.74x0.62mm_HandSolder, F.Cu at (286.0, 101.6)
- added C167: 100nF, Capacitor_SMD:C_0402_1005Metric_Pad0.74x0.62mm_HandSolder, F.Cu at (286.0, 103.6)
- added C168: 100nF, Capacitor_SMD:C_0402_1005Metric_Pad0.74x0.62mm_HandSolder, F.Cu at (286.0, 105.6)
- added C169: 470pF, Capacitor_SMD:C_0402_1005Metric_Pad0.74x0.62mm_HandSolder, F.Cu at (286.0, 107.5)
- added C17: 10nF, Capacitor_SMD:C_0402_1005Metric, F.Cu at (259.0, 57.3)
- added C170: 470pF, Capacitor_SMD:C_0402_1005Metric_Pad0.74x0.62mm_HandSolder, F.Cu at (268.5, 114.2)
- added C171: 7.5pF, Capacitor_SMD:C_0402_1005Metric, F.Cu at (275.2, 101.6)
- added C172: 7.5pF, Capacitor_SMD:C_0402_1005Metric, F.Cu at (275.2, 103.6)
- added C173: 6.2pF, Capacitor_SMD:C_0402_1005Metric, F.Cu at (275.2, 105.6)
- added C174: 470pF, Capacitor_SMD:C_0402_1005Metric, F.Cu at (275.2, 107.5)
- added C175: 470pF, Capacitor_SMD:C_0402_1005Metric, F.Cu at (275.2, 109.5)
- added C176: 1uF, Capacitor_SMD:C_0603_1608Metric, F.Cu at (268.8, 101.9)
- added C177: 470pF, Capacitor_SMD:C_0402_1005Metric, F.Cu at (278.1, 101.6)
- added C178: 470pF, Capacitor_SMD:C_0402_1005Metric, F.Cu at (278.1, 103.6)
- added C179: 1nF, Capacitor_SMD:C_0402_1005Metric, F.Cu at (278.1, 105.6)
- added C18: 100pF, Capacitor_SMD:C_0402_1005Metric, F.Cu at (259.0, 59.3)
- added C180: 10nF, Capacitor_SMD:C_0402_1005Metric, F.Cu at (278.1, 107.5)
- added C181: 10nF, Capacitor_SMD:C_0402_1005Metric, F.Cu at (278.1, 109.5)
- added C182: 13pF, Capacitor_SMD:C_0402_1005Metric, F.Cu at (280.9, 101.6)
- added C183: 68pF, Capacitor_SMD:C_0402_1005Metric, F.Cu at (280.9, 103.6)
- added C184: 68pF, Capacitor_SMD:C_0402_1005Metric, F.Cu at (280.9, 105.6)
- added C185: 470pF, Capacitor_SMD:C_0402_1005Metric, F.Cu at (280.9, 107.5)
- added C186: 12pF, Capacitor_SMD:C_0402_1005Metric, F.Cu at (194.0, 147.0)
- added C187: 1nF, Capacitor_SMD:C_0402_1005Metric, F.Cu at (194.0, 149.0)
- added C188: 12pF, Capacitor_SMD:C_0402_1005Metric, F.Cu at (194.0, 151.0)
- added C189: 1nF, Capacitor_SMD:C_0402_1005Metric, F.Cu at (238.3, 134.6)
- added C19: 470pF, Capacitor_SMD:C_0402_1005Metric, F.Cu at (259.0, 61.2)
- added C190: 100nF, Capacitor_SMD:C_0402_1005Metric, F.Cu at (238.3, 136.5)
- added C191: 100nF, Capacitor_SMD:C_0402_1005Metric, F.Cu at (238.3, 138.5)
- added C192: 1nF, Capacitor_SMD:C_0402_1005Metric, F.Cu at (241.2, 134.6)
- added C193: 1nF, Capacitor_SMD:C_0402_1005Metric, F.Cu at (241.2, 136.5)
- added C194: 1nF, Capacitor_SMD:C_0402_1005Metric, F.Cu at (241.2, 138.5)
- added C195: 470nF, Capacitor_SMD:C_0603_1608Metric, F.Cu at (234.8, 134.8)
- added C196: 1nF, Capacitor_SMD:C_0402_1005Metric, F.Cu at (244.0, 134.6)
- added C197: 470nF, Capacitor_SMD:C_0603_1608Metric, F.Cu at (234.8, 137.3)
- added C198: 100nF, Capacitor_SMD:C_0402_1005Metric, F.Cu at (244.0, 136.5)
- added C199: 1uF, Capacitor_SMD:C_0603_1608Metric, F.Cu at (234.8, 139.8)
- added C2: 1uF, Capacitor_SMD:C_0603_1608Metric, F.Cu at (289.4, 86.9)
- added C20: 470pF, Capacitor_SMD:C_0402_1005Metric, F.Cu at (259.0, 63.2)
- added C200: 1uF, Capacitor_SMD:C_0603_1608Metric, F.Cu at (234.8, 142.4)
- added C201: 1nF, Capacitor_SMD:C_0402_1005Metric, F.Cu at (244.0, 138.5)
- added C202: 22uF, Capacitor_SMD:C_1206_3216Metric, F.Cu at (280.4, 119.3)
- added C203: 10nF, Capacitor_SMD:C_0402_1005Metric, F.Cu at (276.2, 118.6)
- added C204: 22uF, Capacitor_SMD:C_1206_3216Metric, F.Cu at (280.4, 122.6)
- added C205: 10nF, Capacitor_SMD:C_0402_1005Metric, F.Cu at (276.2, 120.6)
- added C206: 100pF, Capacitor_SMD:C_0402_1005Metric, F.Cu at (251.3, 118.6)
- added C207: 100nF, Capacitor_SMD:C_0402_1005Metric, F.Cu at (251.3, 120.6)
- added C208: 22uF, Capacitor_SMD:C_1206_3216Metric, F.Cu at (241.5, 102.3)
- added C209: 22uF, Capacitor_SMD:C_1206_3216Metric, F.Cu at (241.5, 105.7)
- added C21: 100pF, Capacitor_SMD:C_0402_1005Metric, F.Cu at (259.0, 65.2)
- added C210: 1uF, Capacitor_SMD:C_0603_1608Metric, F.Cu at (234.8, 111.8)
- added C211: 1uF, Capacitor_SMD:C_0603_1608Metric, F.Cu at (234.8, 114.3)
- added C212: 100nF, Capacitor_SMD:C_0402_1005Metric, F.Cu at (245.7, 101.6)
- added C213: 100nF, Capacitor_SMD:C_0402_1005Metric, F.Cu at (245.7, 103.6)
- added C214: 100nF, Capacitor_SMD:C_0402_1005Metric, F.Cu at (251.3, 122.5)
- added C215: 100pF, Capacitor_SMD:C_0402_1005Metric, F.Cu at (254.2, 118.6)
- added C216: 1uF, Capacitor_SMD:C_0603_1608Metric, F.Cu at (258.1, 124.8)
- added C217: 100nF, Capacitor_SMD:C_0402_1005Metric, F.Cu at (254.2, 120.6)
- added C218: 100pF, Capacitor_SMD:C_0402_1005Metric, F.Cu at (254.2, 122.5)
- added C219: 1nF, Capacitor_SMD:C_0402_1005Metric, F.Cu at (257.1, 118.6)
- added C22: 10nF, Capacitor_SMD:C_0402_1005Metric, F.Cu at (259.0, 67.2)
- added C220: 1nF, Capacitor_SMD:C_0402_1005Metric, F.Cu at (257.1, 120.6)
- added C221: 1nF, Capacitor_SMD:C_0402_1005Metric, F.Cu at (257.1, 122.5)
- added C222: 100nF, Capacitor_SMD:C_0402_1005Metric, F.Cu at (276.2, 122.5)
- added C223: 18pF, Capacitor_SMD:C_0402_1005Metric, F.Cu at (205.3, 154.9)
- added C224: 30pF, Capacitor_SMD:C_0402_1005Metric, F.Cu at (205.3, 156.9)
- added C225: 18pF, Capacitor_SMD:C_0402_1005Metric, F.Cu at (205.3, 158.9)
- added C226: 7.5pF, Capacitor_SMD:C_0402_1005Metric, F.Cu at (205.3, 162.8)
- added C227: 13pF, Capacitor_SMD:C_0402_1005Metric, F.Cu at (205.3, 164.8)
- added C228: 7.5pF, Capacitor_SMD:C_0402_1005Metric, F.Cu at (205.3, 166.8)
- added C229: 100nF, Capacitor_SMD:C_0402_1005Metric, F.Cu at (276.2, 124.5)
- added C23: 18pF, Capacitor_SMD:C_0402_1005Metric, F.Cu at (254.2, 132.3)
- added C230: 1nF, Capacitor_SMD:C_0402_1005Metric, F.Cu at (280.4, 154.5)
- added C231: 100nF, Capacitor_SMD:C_0402_1005Metric, F.Cu at (280.4, 156.4)
- added C232: 100nF, Capacitor_SMD:C_0402_1005Metric, F.Cu at (280.4, 158.4)
- added C233: 1nF, Capacitor_SMD:C_0402_1005Metric, F.Cu at (280.4, 160.4)
- added C234: 1nF, Capacitor_SMD:C_0402_1005Metric, F.Cu at (188.7, 154.9)
- added C235: 1nF, Capacitor_SMD:C_0402_1005Metric, F.Cu at (188.7, 156.9)
- added C236: 100nF, Capacitor_SMD:C_0402_1005Metric, F.Cu at (276.2, 126.5)
- added C237: 62pF, Capacitor_SMD:C_0402_1005Metric, F.Cu at (222.4, 119.4)
- added C238: 130pF, Capacitor_SMD:C_0402_1005Metric, F.Cu at (222.4, 121.4)
- added C239: 1nF, Capacitor_SMD:C_0402_1005Metric, F.Cu at (222.4, 123.4)
- added C24: 10pF, Capacitor_SMD:C_0402_1005Metric, F.Cu at (254.2, 134.3)
- added C240: 100pF, Capacitor_SMD:C_0402_1005Metric, F.Cu at (222.4, 125.3)
- added C241: 100nF, Capacitor_SMD:C_0402_1005Metric, F.Cu at (222.4, 127.3)
- added C242: 1nF, Capacitor_SMD:C_0402_1005Metric, F.Cu at (222.4, 129.3)
- added C243: 91pF, Capacitor_SMD:C_0402_1005Metric, F.Cu at (222.4, 131.2)
- added C244: C, Capacitor_SMD:C_0402_1005Metric, F.Cu at (222.4, 133.2)
- added C245: 27pF, Capacitor_SMD:C_0402_1005Metric, F.Cu at (222.4, 137.2)
- added C246: C, Capacitor_SMD:C_0402_1005Metric, F.Cu at (222.4, 139.2)
- added C247: 1nF, Capacitor_SMD:C_0402_1005Metric, F.Cu at (222.4, 141.1)
- added C248: 100pF, Capacitor_SMD:C_0402_1005Metric, F.Cu at (222.4, 143.1)
- added C249: 100nF, Capacitor_SMD:C_0402_1005Metric, F.Cu at (222.4, 145.1)
- added C25: 6.8pF, Capacitor_SMD:C_0402_1005Metric, F.Cu at (254.2, 136.2)
- added C250: 1nF, Capacitor_SMD:C_0402_1005Metric, F.Cu at (222.4, 147.0)
- added C251: C, Capacitor_SMD:C_0402_1005Metric, F.Cu at (222.4, 149.0)
- added C252: 24pF, Capacitor_SMD:C_0402_1005Metric, F.Cu at (222.4, 151.0)
- added C253: C, Capacitor_SMD:C_0402_1005Metric, F.Cu at (213.5, 137.2)
- added C254: C, Capacitor_SMD:C_0402_1005Metric, F.Cu at (213.5, 139.2)
- added C255: 100pF, Capacitor_SMD:C_0402_1005Metric, F.Cu at (213.5, 141.1)
- added C256: 10nF, Capacitor_SMD:C_0402_1005Metric, F.Cu at (213.5, 143.1)
- added C257: 1nF, Capacitor_SMD:C_0402_1005Metric, F.Cu at (213.5, 145.1)
- added C258: 1nF, Capacitor_SMD:C_0402_1005Metric, F.Cu at (213.5, 147.0)
- added C259: C, Capacitor_SMD:C_0402_1005Metric, F.Cu at (213.5, 149.0)
- added C26: 8.2pF, Capacitor_SMD:C_0402_1005Metric, F.Cu at (254.2, 138.2)
- added C260: C, Capacitor_SMD:C_0402_1005Metric, F.Cu at (213.5, 151.0)
- added C261: C, Capacitor_SMD:C_0402_1005Metric, F.Cu at (213.5, 119.4)
- added C262: C, Capacitor_SMD:C_0402_1005Metric, F.Cu at (213.5, 121.4)
- added C263: 1nF, Capacitor_SMD:C_0402_1005Metric, F.Cu at (213.5, 123.4)
- added C264: 100pF, Capacitor_SMD:C_0402_1005Metric, F.Cu at (213.5, 125.3)
- added C265: 1nF, Capacitor_SMD:C_0402_1005Metric, F.Cu at (213.5, 127.3)
- added C266: 10nF, Capacitor_SMD:C_0402_1005Metric, F.Cu at (213.5, 129.3)
- added C267: C, Capacitor_SMD:C_0402_1005Metric, F.Cu at (213.5, 131.2)
- added C268: C, Capacitor_SMD:C_0402_1005Metric, F.Cu at (213.5, 133.2)
- added C269: 22pF, Capacitor_SMD:C_0402_1005Metric, F.Cu at (269.8, 164.4)
- added C27: 36pF, Capacitor_SMD:C_0402_1005Metric, F.Cu at (254.2, 140.2)
- added C270: 39pF, Capacitor_SMD:C_0402_1005Metric, F.Cu at (269.8, 166.3)
- added C271: 39pF, Capacitor_SMD:C_0402_1005Metric, F.Cu at (269.8, 168.3)
- added C272: 22pF, Capacitor_SMD:C_0402_1005Metric, F.Cu at (269.8, 170.3)
- added C273: 8.2pF, Capacitor_SMD:C_0402_1005Metric, F.Cu at (290.9, 154.5)
- added C274: 15pF, Capacitor_SMD:C_0402_1005Metric, F.Cu at (290.9, 156.4)
- added C275: 15pF, Capacitor_SMD:C_0402_1005Metric, F.Cu at (290.9, 158.4)
- added C276: 8.2pF, Capacitor_SMD:C_0402_1005Metric, F.Cu at (290.9, 160.4)
- added C277: 100pF, Capacitor_SMD:C_0402_1005Metric, F.Cu at (244.8, 57.3)
- added C278: 10nF, Capacitor_SMD:C_0402_1005Metric, F.Cu at (244.8, 59.3)
- added C279: 470pF, Capacitor_SMD:C_0402_1005Metric, F.Cu at (244.8, 61.2)
- added C28: 91pF, Capacitor_SMD:C_0402_1005Metric, F.Cu at (263.6, 118.6)
- added C280: 100pF, Capacitor_SMD:C_0402_1005Metric, F.Cu at (244.8, 63.2)
- added C281: 10nF, Capacitor_SMD:C_0402_1005Metric, F.Cu at (244.8, 65.2)
- added C282: 470pF, Capacitor_SMD:C_0402_1005Metric, F.Cu at (244.8, 67.2)
- added C283: 10pF, Capacitor_SMD:C_0402_1005Metric, F.Cu at (250.6, 101.6)
- added C284: 100nF, Capacitor_SMD:C_0402_1005Metric, F.Cu at (250.6, 103.6)
- added C285: 10pF, Capacitor_SMD:C_0402_1005Metric, F.Cu at (250.6, 105.6)
- added C286: 100nF, Capacitor_SMD:C_0402_1005Metric, F.Cu at (250.6, 107.5)
- added C287: 10pF, Capacitor_SMD:C_0402_1005Metric, F.Cu at (250.6, 109.5)
- added C288: 100nF, Capacitor_SMD:C_0402_1005Metric, F.Cu at (250.6, 111.5)
- added C289: 100nF, Capacitor_SMD:C_0402_1005Metric, F.Cu at (253.5, 101.6)
- added C29: 4.3pF, Capacitor_SMD:C_0402_1005Metric, F.Cu at (263.6, 120.6)
- added C290: 100nF, Capacitor_SMD:C_0402_1005Metric, F.Cu at (253.5, 103.6)
- added C291: 100nF, Capacitor_SMD:C_0402_1005Metric, F.Cu at (253.5, 105.6)
- added C292: 100nF, Capacitor_SMD:C_0402_1005Metric, F.Cu at (253.5, 107.5)
- added C293: 100nF, Capacitor_SMD:C_0402_1005Metric, F.Cu at (253.5, 109.5)
- added C294: 58.3nF, Capacitor_SMD:C_0402_1005Metric, F.Cu at (253.5, 111.5)
- added C295: 793nF, Capacitor_SMD:C_0603_1608Metric, F.Cu at (259.8, 101.9)
- added C296: 100nF, Capacitor_SMD:C_0402_1005Metric, F.Cu at (256.4, 101.6)
- added C297: 100nF, Capacitor_SMD:C_0402_1005Metric, F.Cu at (256.4, 103.6)
- added C298: 26.6nF, Capacitor_SMD:C_0402_1005Metric, F.Cu at (256.4, 105.6)
- added C3: 100nF, Capacitor_SMD:C_0402_1005Metric, F.Cu at (293.6, 84.0)
- added C30: 160pF, Capacitor_SMD:C_0402_1005Metric, F.Cu at (263.6, 122.5)
- added C301: 47nF, Capacitor_SMD:C_0402_1005Metric, F.Cu at (224.5, 101.6)
- added C302: 47nF, Capacitor_SMD:C_0402_1005Metric, F.Cu at (224.5, 103.6)
- added C303: 4.7uF, Capacitor_SMD:C_0603_1608Metric, F.Cu at (214.1, 101.9)
- added C304: 1nF, Capacitor_SMD:C_0402_1005Metric, F.Cu at (224.5, 105.6)
- added C305: 10uF, Capacitor_SMD:C_0603_1608Metric, F.Cu at (214.1, 104.4)
- added C306: 100nF, Capacitor_SMD:C_0402_1005Metric, F.Cu at (224.5, 107.5)
- added C307: 10uF, Capacitor_SMD:C_0603_1608Metric, F.Cu at (214.1, 106.9)
- added C308: 10uF, Capacitor_SMD:C_0603_1608Metric, F.Cu at (214.1, 109.4)
- added C309: 10uF, Capacitor_SMD:C_0603_1608Metric, F.Cu at (214.1, 111.9)
- added C31: 4.3pF, Capacitor_SMD:C_0402_1005Metric, F.Cu at (263.6, 124.5)
- added C310: 10uF, Capacitor_SMD:C_0603_1608Metric, F.Cu at (214.1, 114.4)
- added C311: 10uF, Capacitor_SMD:C_0603_1608Metric, F.Cu at (218.1, 101.9)
- added C312: 10uF, Capacitor_SMD:C_0603_1608Metric, F.Cu at (218.1, 104.4)
- added C313: 0.47uF, Capacitor_SMD:C_0603_1608Metric, F.Cu at (259.7, 149.0)
- added C314: 0.47uF, Capacitor_SMD:C_0603_1608Metric, F.Cu at (259.7, 151.5)
- added C315: 100nF, Capacitor_SMD:C_0402_1005Metric, F.Cu at (264.9, 144.2)
- added C316: 2.2uF, Capacitor_SMD:C_0603_1608Metric, F.Cu at (200.0, 95.8)
- added C317: 2.2uF, Capacitor_SMD:C_0603_1608Metric, F.Cu at (200.0, 98.3)
- added C318: 100nF, Capacitor_SMD:C_0402_1005Metric, F.Cu at (189.9, 114.1)
- added C319: 100nF, Capacitor_SMD:C_0402_1005Metric, F.Cu at (189.9, 116.0)
- added C32: 91pF, Capacitor_SMD:C_0402_1005Metric, F.Cu at (263.6, 126.5)
- added C320: 100nF, Capacitor_SMD:C_0402_1005Metric, F.Cu at (189.9, 118.0)
- added C321: 100nF, Capacitor_SMD:C_0402_1005Metric, F.Cu at (189.9, 120.0)
- added C322: 18pF, Capacitor_SMD:C_0402_1005Metric, F.Cu at (189.9, 121.9)
- added C323: 18pF, Capacitor_SMD:C_0402_1005Metric, F.Cu at (192.8, 114.1)
- added C324: 18pF, Capacitor_SMD:C_0402_1005Metric, F.Cu at (192.8, 116.0)
- added C325: 18pF, Capacitor_SMD:C_0402_1005Metric, F.Cu at (192.8, 118.0)
- added C326: 100nF, Capacitor_SMD:C_0402_1005Metric, F.Cu at (192.8, 120.0)
- added C327: 100nF, Capacitor_SMD:C_0402_1005Metric, F.Cu at (192.8, 121.9)
- added C328: 100nF, Capacitor_SMD:C_0402_1005Metric, F.Cu at (195.7, 114.1)
- added C329: 100nF, Capacitor_SMD:C_0402_1005Metric, F.Cu at (195.7, 116.0)
- added C33: 470pF, Capacitor_SMD:C_0402_1005Metric, F.Cu at (269.8, 144.2)
- added C330: 100nF, Capacitor_SMD:C_0402_1005Metric, F.Cu at (195.7, 118.0)
- added C331: 100nF, Capacitor_SMD:C_0402_1005Metric, F.Cu at (195.7, 120.0)
- added C332: 1uF, Capacitor_SMD:C_0603_1608Metric, F.Cu at (200.0, 100.8)
- added C333: 10nF, Capacitor_SMD:C_0402_1005Metric, F.Cu at (288.3, 63.3)
- added C334: 10nF, Capacitor_SMD:C_0402_1005Metric, F.Cu at (288.3, 65.2)
- added C335: 10nF, Capacitor_SMD:C_0402_1005Metric, F.Cu at (288.3, 67.2)
- added C336: 10nF, Capacitor_SMD:C_0402_1005Metric, F.Cu at (254.2, 156.2)
- added C337: 10nF, Capacitor_SMD:C_0402_1005Metric, F.Cu at (254.2, 158.2)
- added C338: 10nF, Capacitor_SMD:C_0402_1005Metric, F.Cu at (254.2, 160.1)
- added C339: 10nF, Capacitor_SMD:C_0402_1005Metric, F.Cu at (188.7, 164.9)
- added C34: 470pF, Capacitor_SMD:C_0402_1005Metric, F.Cu at (269.8, 146.1)
- added C340: 100nF, Capacitor_SMD:C_0402_1005Metric, F.Cu at (188.7, 166.8)
- added C341: 100nF, Capacitor_SMD:C_0402_1005Metric, F.Cu at (221.3, 163.6)
- added C342: 100nF, Capacitor_SMD:C_0402_1005Metric, F.Cu at (221.3, 165.6)
- added C343: 100nF, Capacitor_SMD:C_0402_1005Metric, F.Cu at (220.4, 88.5)
- added C344: 100nF, Capacitor_SMD:C_0402_1005Metric, F.Cu at (220.4, 90.5)
- added C345: 10uF, Capacitor_SMD:C_0603_1608Metric, F.Cu at (214.1, 82.3)
- added C346: 10uF, Capacitor_SMD:C_0603_1608Metric, F.Cu at (214.1, 84.8)
- added C347: 10uF, Capacitor_SMD:C_0603_1608Metric, F.Cu at (214.1, 87.3)
- added C348: 10uF, Capacitor_SMD:C_0603_1608Metric, F.Cu at (214.1, 89.8)
- added C349: 100nF, Capacitor_SMD:C_0402_1005Metric, F.Cu at (220.4, 92.5)
- added C35: 100pF, Capacitor_SMD:C_0402_1005Metric, F.Cu at (269.8, 148.1)
- added C350: 1uF, Capacitor_SMD:C_0603_1608Metric, F.Cu at (214.1, 92.4)
- added C351: 1uF, Capacitor_SMD:C_0603_1608Metric, F.Cu at (214.1, 94.9)
- added C352: 1uF, Capacitor_SMD:C_0603_1608Metric, F.Cu at (214.1, 97.4)
- added C353: 10uF, Capacitor_SMD:C_0603_1608Metric, F.Cu at (283.8, 164.6)
- added C354: 100nF, Capacitor_SMD:C_0402_1005Metric, F.Cu at (280.4, 164.3)
- added C355: 100nF, Capacitor_SMD:C_0402_1005Metric, F.Cu at (280.4, 166.3)
- added C356: 100nF, Capacitor_SMD:C_0402_1005Metric, F.Cu at (280.4, 168.3)
- added C357: 4.7nF, Capacitor_SMD:C_0402_1005Metric, F.Cu at (280.4, 170.2)
- added C358: 1uF, Capacitor_SMD:C_0603_1608Metric, F.Cu at (283.8, 167.1)
- added C359: 1uF, Capacitor_SMD:C_0603_1608Metric, F.Cu at (283.8, 169.6)
- added C36: 100nF, Capacitor_SMD:C_0402_1005Metric, F.Cu at (269.8, 150.1)
- added C360: 22uF, Capacitor_SMD:C_1206_3216Metric, F.Cu at (271.2, 155.2)
- added C361: 22uF, Capacitor_SMD:C_1206_3216Metric, F.Cu at (271.2, 158.5)
- added C362: 10nF, Capacitor_SMD:C_0402_1005Metric, F.Cu at (275.5, 158.4)
- added C363: 10nF, Capacitor_SMD:C_0402_1005Metric, F.Cu at (275.5, 160.4)
- added C364: 15pF, Capacitor_SMD:C_0402_1005Metric, F.Cu at (213.5, 57.3)
- added C365: 15pF, Capacitor_SMD:C_0402_1005Metric, F.Cu at (213.5, 59.3)
- added C366: 4.7uF, Capacitor_SMD:C_0603_1608Metric, F.Cu at (220.5, 57.6)
- added C367: 4.7uF, Capacitor_SMD:C_0603_1608Metric, F.Cu at (220.5, 60.1)
- added C368: 4.7uF, Capacitor_SMD:C_0603_1608Metric, F.Cu at (220.5, 62.6)
- added C369: 100nF, Capacitor_SMD:C_0402_1005Metric, F.Cu at (213.5, 61.2)
- added C37: 82pF, Capacitor_SMD:C_0402_1005Metric, F.Cu at (183.8, 154.9)
- added C370: 100nF, Capacitor_SMD:C_0402_1005Metric, F.Cu at (213.5, 63.2)
- added C371: 4.7uF, Capacitor_SMD:C_0603_1608Metric, F.Cu at (220.5, 65.1)
- added C372: 100nF, Capacitor_SMD:C_0402_1005Metric, F.Cu at (213.5, 65.2)
- added C373: 100nF, Capacitor_SMD:C_0402_1005Metric, F.Cu at (213.5, 67.2)
- added C374: 100nF, Capacitor_SMD:C_0402_1005Metric, F.Cu at (213.5, 69.1)
- added C375: 100nF, Capacitor_SMD:C_0402_1005Metric, F.Cu at (213.5, 71.1)
- added C376: 100pF, Capacitor_SMD:C_0402_1005Metric, F.Cu at (259.1, 132.3)
- added C377: 10nF, Capacitor_SMD:C_0402_1005Metric, F.Cu at (259.1, 134.3)
- added C378: 10nF, Capacitor_SMD:C_0402_1005Metric, F.Cu at (259.1, 136.2)
- added C379: 100pF, Capacitor_SMD:C_0402_1005Metric, F.Cu at (259.1, 138.2)
- added C38: 5.1pF, Capacitor_SMD:C_0402_1005Metric, F.Cu at (183.8, 156.9)
- added C380: 10nF, Capacitor_SMD:C_0402_1005Metric, F.Cu at (259.1, 140.2)
- added C381: 10uF, Capacitor_SMD:C_0603_1608Metric, F.Cu at (218.1, 106.9)
- added C382: 10uF, Capacitor_SMD:C_0603_1608Metric, F.Cu at (218.1, 109.4)
- added C383: 10uF, Capacitor_SMD:C_0603_1608Metric, F.Cu at (218.1, 111.9)
- added C384: 100nF, Capacitor_SMD:C_0402_1005Metric, F.Cu at (224.5, 109.5)
- added C39: 82pF, Capacitor_SMD:C_0402_1005Metric, F.Cu at (183.8, 158.9)
- added C4: 10uF, Capacitor_SMD:C_0603_1608Metric, F.Cu at (292.2, 126.5)
- added C40: 470pF, Capacitor_SMD:C_0402_1005Metric, F.Cu at (259.1, 166.3)
- added C41: 100nF, Capacitor_SMD:C_0402_1005Metric, F.Cu at (259.1, 168.2)
- added C42: 100nF, Capacitor_SMD:C_0402_1005Metric, F.Cu at (259.1, 170.2)
- added C43: 470pF, Capacitor_SMD:C_0402_1005Metric, F.Cu at (259.1, 172.2)
- added C44: 3.64nF, Capacitor_SMD:C_0402_1005Metric, F.Cu at (268.2, 57.3)
- added C45: 46.5nF, Capacitor_SMD:C_0402_1005Metric, F.Cu at (268.2, 59.3)
- added C46: 1.66nF, Capacitor_SMD:C_0402_1005Metric, F.Cu at (268.2, 61.2)
- added C47: 100nF, Capacitor_SMD:C_0402_1005Metric, F.Cu at (268.2, 63.2)
- added C48: 100nF, Capacitor_SMD:C_0402_1005Metric, F.Cu at (268.2, 65.2)
- added C49: 100nF, Capacitor_SMD:C_0402_1005Metric, F.Cu at (268.2, 67.2)
- added C5: 100nF, Capacitor_SMD:C_0402_1005Metric, F.Cu at (286.7, 126.9)
- added C50: 100nF, Capacitor_SMD:C_0402_1005Metric, F.Cu at (271.0, 57.3)
- added C51: 100nF, Capacitor_SMD:C_0402_1005Metric, F.Cu at (271.0, 59.3)
- added C52: 10pF, Capacitor_SMD:C_0402_1005Metric, F.Cu at (271.0, 61.2)
- added C53: 100nF, Capacitor_SMD:C_0402_1005Metric, F.Cu at (271.0, 63.2)
- added C54: 10pF, Capacitor_SMD:C_0402_1005Metric, F.Cu at (271.0, 65.2)
- added C55: 100nF, Capacitor_SMD:C_0402_1005Metric, F.Cu at (271.0, 67.2)
- added C56: 10pF, Capacitor_SMD:C_0402_1005Metric, F.Cu at (273.9, 57.3)
- added C57: 100nF, Capacitor_SMD:C_0402_1005Metric, F.Cu at (273.9, 59.3)
- added C58: 100nF, Capacitor_SMD:C_0402_1005Metric, F.Cu at (273.9, 61.2)
- added C59: 100nF, Capacitor_SMD:C_0402_1005Metric, F.Cu at (273.9, 63.2)
- added C6: 22uF, Capacitor_SMD:C_0805_2012Metric, F.Cu at (292.4, 123.7)
- added C60: 1nF, Capacitor_SMD:C_0402_1005Metric, F.Cu at (273.9, 65.2)
- added C61: 1nF, Capacitor_SMD:C_0402_1005Metric, F.Cu at (273.9, 67.2)
- added C62: 11pF, Capacitor_SMD:C_0402_1005Metric, F.Cu at (276.8, 57.3)
- added C63: 11pF, Capacitor_SMD:C_0402_1005Metric, F.Cu at (276.8, 59.3)
- added C64: 11pF, Capacitor_SMD:C_0402_1005Metric, F.Cu at (276.8, 61.2)
- added C65: 11pF, Capacitor_SMD:C_0402_1005Metric, F.Cu at (276.8, 63.2)
- added C66: 100nF, Capacitor_SMD:C_0402_1005Metric, F.Cu at (288.8, 95.6)
- added C67: 10pF, Capacitor_SMD:C_0402_1005Metric, F.Cu at (244.0, 82.0)
- added C68: 100nF, Capacitor_SMD:C_0402_1005Metric, F.Cu at (244.0, 84.0)
- added C69: 10pF, Capacitor_SMD:C_0402_1005Metric, F.Cu at (244.0, 86.0)
- added C7: 100nF, Capacitor_SMD:C_0402_1005Metric, F.Cu at (288.3, 136.6)
- added C70: 100nF, Capacitor_SMD:C_0402_1005Metric, F.Cu at (244.0, 88.0)
- added C71: 10pF, Capacitor_SMD:C_0402_1005Metric, F.Cu at (244.0, 89.9)
- added C72: 100nF, Capacitor_SMD:C_0402_1005Metric, F.Cu at (244.0, 91.9)
- added C73: 100nF, Capacitor_SMD:C_0402_1005Metric, F.Cu at (244.0, 93.9)
- added C74: 100nF, Capacitor_SMD:C_0402_1005Metric, F.Cu at (246.9, 82.0)
- added C75: 100nF, Capacitor_SMD:C_0402_1005Metric, F.Cu at (246.9, 84.0)
- added C76: 100nF, Capacitor_SMD:C_0402_1005Metric, F.Cu at (246.9, 86.0)
- added C77: 100nF, Capacitor_SMD:C_0402_1005Metric, F.Cu at (246.9, 88.0)
- added C78: 58.3nF, Capacitor_SMD:C_0402_1005Metric, F.Cu at (246.9, 89.9)
- added C79: 100nF, Capacitor_SMD:C_0402_1005Metric, F.Cu at (246.9, 91.9)
- added C8: 22uF, Capacitor_SMD:C_0805_2012Metric, F.Cu at (281.7, 137.1)
- added C80: 100nF, Capacitor_SMD:C_0402_1005Metric, F.Cu at (246.9, 93.9)
- added C81: 793nF, Capacitor_SMD:C_0603_1608Metric, F.Cu at (256.1, 82.3)
- added C82: 1nF, Capacitor_SMD:C_0402_1005Metric, F.Cu at (249.7, 82.0)
- added C83: 1nF, Capacitor_SMD:C_0402_1005Metric, F.Cu at (249.7, 84.0)
- added C84: 26.6nF, Capacitor_SMD:C_0402_1005Metric, F.Cu at (249.7, 86.0)
- added C85: 5.1pH, Capacitor_SMD:C_0402_1005Metric, F.Cu at (249.7, 88.0)
- added C86: 5.1pH, Capacitor_SMD:C_0402_1005Metric, F.Cu at (249.7, 89.9)
- added C87: 5.1pH, Capacitor_SMD:C_0402_1005Metric, F.Cu at (249.7, 91.9)
- added C88: 5.1pH, Capacitor_SMD:C_0402_1005Metric, F.Cu at (249.7, 93.9)
- added C89: 470pF, Capacitor_SMD:C_0402_1005Metric, F.Cu at (230.5, 82.0)
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
Commit message: :3
Parts:
- removed C1, C10, C111, C112, C114, C129, C133, C134, C135, C136, C137, C138, C14, C145, C15, C156, C158, C159, C162, C190, C191, C198, C207, C212, C213, C214, C217, C222, C229, C231, C232, C236, C241, C249, C284, C286, C288, C289, C290, C291, C292, C293, C296, C297, C3, C306, C315, C318, C319, C320, C321, C326, C327, C328, C329, C330, C331, C340, C341, C342, C343, C344, C349, C354, C355, C356, C36, C369, C370, C372, C373, C374, C375, C384, C41, C42, C47, C48, C49, C5, C50, C51, C53, C55, C57, C58, C59, C66, C68, C7, C70, C72, C73, C74, C75, C76, C77, C79, C80: 100nF, Capacitor_SMD:C_0402_1005Metric
- removed C100, C101, C123, C183, C184: 68pF, Capacitor_SMD:C_0402_1005Metric
- removed C102, C126, C127, C16, C174, C175, C177, C178, C185, C19, C20, C279, C282, C33, C34, C40, C43, C89, C90, C91, C92, C96: 470pF, Capacitor_SMD:C_0402_1005Metric
- removed C103, C105, C108, C109, C110, C113, C115, C116, C179, C187, C189, C192, C193, C194, C196, C201, C219, C220, C221, C230, C233, C234, C235, C239, C242, C247, C250, C257, C258, C263, C265, C304, C60, C61, C82, C83: 1nF, Capacitor_SMD:C_0402_1005Metric
- removed C104, C11, C119, C120, C148, C149, C150, C151, C152, C153, C157, C163, C164, C165, C176, C199, C2, C200, C210, C211, C216, C332, C350, C351, C352, C358, C359: 1uF, Capacitor_SMD:C_0603_1608Metric
- removed C106, C107, C186, C188: 12pF, Capacitor_SMD:C_0402_1005Metric
- removed C117, C118, C195, C197: 470nF, Capacitor_SMD:C_0603_1608Metric
- removed C12, C13, C316, C317: 2.2uF, Capacitor_SMD:C_0603_1608Metric
- removed C121, C125, C270, C271: 39pF, Capacitor_SMD:C_0402_1005Metric
- removed C122, C124: 1.1pF, Capacitor_SMD:C_0402_1005Metric
- removed C128, C140, C143, C18, C206, C21, C215, C218, C240, C248, C255, C264, C277, C280, C35, C376, C379: 100pF, Capacitor_SMD:C_0402_1005Metric
- removed C130, C132, C27: 36pF, Capacitor_SMD:C_0402_1005Metric
- removed C131: 1.3pF, Capacitor_SMD:C_0402_1005Metric
- removed C139, C141, C142, C144, C237: 62pF, Capacitor_SMD:C_0402_1005Metric
- removed C146, C147, C155, C161: 4.7pF, Capacitor_SMD:C_0402_1005Metric
- removed C154, C160, C24, C283, C285, C287, C52, C54, C56, C67, C69, C71: 10pF, Capacitor_SMD:C_0402_1005Metric
- removed C166, C169, C170: 470pF, Capacitor_SMD:C_0402_1005Metric_Pad0.74x0.62mm_HandSolder
- removed C167, C168: 100nF, Capacitor_SMD:C_0402_1005Metric_Pad0.74x0.62mm_HandSolder
- removed C17, C180, C181, C203, C205, C22, C256, C266, C278, C281, C333, C334, C335, C336, C337, C338, C339, C362, C363, C377, C378, C380, C97, C98: 10nF, Capacitor_SMD:C_0402_1005Metric
- removed C171, C172, C226, C228: 7.5pF, Capacitor_SMD:C_0402_1005Metric
- removed C173: 6.2pF, Capacitor_SMD:C_0402_1005Metric
- removed C182, C227, C99: 13pF, Capacitor_SMD:C_0402_1005Metric
- removed C202, C204, C208, C209, C360, C361: 22uF, Capacitor_SMD:C_1206_3216Metric
- removed C223, C225, C23, C322, C323, C324, C325, C93: 18pF, Capacitor_SMD:C_0402_1005Metric
- removed C224: 30pF, Capacitor_SMD:C_0402_1005Metric
- removed C238: 130pF, Capacitor_SMD:C_0402_1005Metric
- removed C243, C28, C32: 91pF, Capacitor_SMD:C_0402_1005Metric
- removed C244, C246, C251, C253, C254, C259, C260, C261, C262, C267, C268: C, Capacitor_SMD:C_0402_1005Metric
- removed C245: 27pF, Capacitor_SMD:C_0402_1005Metric
- removed C25: 6.8pF, Capacitor_SMD:C_0402_1005Metric
- removed C252: 24pF, Capacitor_SMD:C_0402_1005Metric
- removed C26, C273, C276: 8.2pF, Capacitor_SMD:C_0402_1005Metric
- removed C269, C272: 22pF, Capacitor_SMD:C_0402_1005Metric
- removed C274, C275, C364, C365: 15pF, Capacitor_SMD:C_0402_1005Metric
- removed C29, C31: 4.3pF, Capacitor_SMD:C_0402_1005Metric
- removed C294, C78: 58.3nF, Capacitor_SMD:C_0402_1005Metric
- removed C295, C81: 793nF, Capacitor_SMD:C_0603_1608Metric
- removed C298, C84: 26.6nF, Capacitor_SMD:C_0402_1005Metric
- removed C30: 160pF, Capacitor_SMD:C_0402_1005Metric
- removed C301, C302: 47nF, Capacitor_SMD:C_0402_1005Metric
- removed C303, C366, C367, C368, C371: 4.7uF, Capacitor_SMD:C_0603_1608Metric
- removed C305, C307, C308, C309, C310, C311, C312, C345, C346, C347, C348, C353, C381, C382, C383, C4, C9: 10uF, Capacitor_SMD:C_0603_1608Metric
- removed C313, C314: 0.47uF, Capacitor_SMD:C_0603_1608Metric
- removed C357: 4.7nF, Capacitor_SMD:C_0402_1005Metric
- removed C37, C39: 82pF, Capacitor_SMD:C_0402_1005Metric
- removed C38: 5.1pF, Capacitor_SMD:C_0402_1005Metric
- removed C44: 3.64nF, Capacitor_SMD:C_0402_1005Metric
- removed C45: 46.5nF, Capacitor_SMD:C_0402_1005Metric
- removed C46: 1.66nF, Capacitor_SMD:C_0402_1005Metric
- removed C6, C8: 22uF, Capacitor_SMD:C_0805_2012Metric
- removed C62, C63, C64, C65: 11pF, Capacitor_SMD:C_0402_1005Metric
- removed C85, C86, C87, C88: 5.1pH, Capacitor_SMD:C_0402_1005Metric
- removed C94, C95: 16pF, Capacitor_SMD:C_0402_1005Metric
- removed D1, D2: BAV99, Package_TO_SOT_SMD:SOT-23
- removed D10, D11, D13, D14, D15, D17, D18, D19, D21, D22, D23, D5, D6, D7, D9: D, Diode_SMD:D_SOD-523
- removed D3: TPD2E001DRLR, easyeda2kicad:SOT-553-5_L1.6-W1.2-P0.50-LS1.6-BR
- removed D4: SMAJ5.0A, Diode_SMD:D_SMA
- removed D8: RCLAMP0531T.TCT, easyeda2kicad:SLP1006P2T_L1.0-W0.6-P0.65-L
- removed F1: MF-MSMF150-2, Fuse:Fuse_1812_4532Metric
- removed FB1: FerriteBead, Inductor_SMD:L_0402_1005Metric
- removed FPC1: FPC-05F-14PH15, easyeda2kicad:FPC-SMD_14P-P0.50_XUNPU_FPC-05F-14PH15
- removed J2, J3: Conn_ARM_SWD_TagConnect_TC2030, Connector:Tag-Connect_TC2030-IDC-FP_2x03_P1.27mm_Vertical
- removed L1: 2.2uH, Inductor_SMD:L_1008_2520Metric
- removed L10: 30nH, Inductor_SMD:L_0402_1005Metric
- removed L100: AOTA-B201610S3R3-101-T, easyeda2kicad:IND-SMD_L2.0-W1.6_AOTA-B201610S3R3-101-T
- removed L11, L15, L17, L19: 13nH, Inductor_SMD:L_0402_1005Metric
- removed L12, L14, L20, L21, L24, L25, L32, L33, L58, L59, L71, L97, L98: 270nH, Inductor_SMD:L_0603_1608Metric
- removed L13: 7.5nH, Inductor_SMD:L_0402_1005Metric
- removed L16, L3, L4, L46, L5, L73, L74, L77, L78, L81, L82, L85, L86, L94, L95, L96: 470nH, Inductor_SMD:L_0603_1608Metric
- removed L18: 220nH, Inductor_SMD:L_0402_1005Metric
- removed L2: 1.5uH, Inductor_SMD:L_1008_2520Metric
- removed L22, L23: 51nH, Inductor_SMD:L_0402_1005Metric
- removed L26, L27, L72: 27nH, Inductor_SMD:L_0402_1005Metric
- removed L28, L29, L75: 12nH, Inductor_SMD:L_0402_1005Metric
- removed L30, L31, L7: 39nH, Inductor_SMD:L_0402_1005Metric
- removed L34, L35, L60, L61: 390nH, Inductor_SMD:L_0603_1608Metric
- removed L36, L37: 180nH, Inductor_SMD:L_0603_1608Metric
- removed L38, L39, L64, L65: 750nH, Inductor_SMD:L_0805_2012Metric
- removed L40, L66: HCCF2-455.000-LTWCDL, easyeda2kicad:FILTER-SMD_4P-L11.9-W6.5-P5.50-LS7.5-BL
- removed L41, L45: 3.3nH, Inductor_SMD:L_0402_1005Metric
- removed L42, L44: 120nH, Inductor_SMD:L_0402_1005Metric
- removed L43: 2nH, Inductor_SMD:L_0402_1005Metric
- removed L47, L49, L56, L57: 3.6nH, Inductor_SMD:L_0402_1005Metric
- removed L48: 100nH, Inductor_SMD:L_0402_1005Metric
- removed L50, L51, L52, L53, L62, L63: 180nH, Inductor_SMD:L_0402_1005Metric
- removed L54, L55: 18nH, Inductor_SMD:L_0402_1005Metric
- removed L6: 43nH, Inductor_SMD:L_0402_1005Metric
- removed L67, L68: 56nH, Inductor_SMD:L_0402_1005Metric
- removed L69, L70: 22nH, Inductor_SMD:L_0402_1005Metric
- removed L76: 4.7nH, Inductor_SMD:L_0402_1005Metric
- removed L79: 4.3nH, Inductor_SMD:L_0402_1005Metric
- removed L8: 8.2nH, Inductor_SMD:L_0402_1005Metric
- removed L9: 16nH, Inductor_SMD:L_0402_1005Metric
- removed L99: 1uH, Inductor_SMD:L_1008_2520Metric
- removed Q1, Q10, Q11, Q13, Q2, Q3: MMBT2222A, Package_TO_SOT_SMD:SOT-23
- removed Q12, Q14, Q4, Q5: BSS84, Package_TO_SOT_SMD:SOT-23
- removed Q15, Q16: 2N7002, Package_TO_SOT_SMD:SOT-23
- removed Q6, Q7: AFT05MS004NT1, easyeda2kicad:SOT-89-3_L4.5-W2.5-P1.50-LS4.2-BR
- removed R1: 33.2k, Resistor_SMD:R_0402_1005Metric
- removed R10, R103, R104, R105, R106, R107, R108, R109, R110, R112, R113, R114, R115, R12, R123, R13, R2, R38, R39, R4, R42, R43, R49, R50, R51, R52, R82, R83, R85, TH1: 10k, Resistor_SMD:R_0402_1005Metric
- removed R100: 30.31k, Resistor_SMD:R_0402_1005Metric
- removed R101, R55, R56: 50, Resistor_SMD:R_0402_1005Metric
- removed R102: 0.01, Resistor_SMD:R_0805_2012Metric
- removed R11, R116, R117, R118, R37, R40, R44, R45, R70, R72, R73, R74, R75, R76, R77, R78, R79, R8, R80, R81, R84, R9: 1k, Resistor_SMD:R_0402_1005Metric
- removed R111: 6.8, Resistor_SMD:R_0603_1608Metric
- removed R119, R120, R61, R62: 160, Resistor_SMD:R_0402_1005Metric
- removed R121, R122, R26, R27, R57, R58: 2.2k, Resistor_SMD:R_0402_1005Metric
- removed R124: 33, Resistor_SMD:R_0402_1005Metric
- removed R125, R126: 0, Resistor_SMD:R_0402_1005Metric
- removed R14, R16, R18, R19, R28, R30, R31, R33, R34, R36: 300, Resistor_SMD:R_0402_1005Metric
- removed R15, R29: 18, Resistor_SMD:R_0402_1005Metric
- removed R17, R21, R86: 5.1k, Resistor_SMD:R_0402_1005Metric
- removed R20: 1.84k, Resistor_SMD:R_0402_1005Metric
- removed R22, R87: 56.3, Resistor_SMD:R_0402_1005Metric
- removed R23, R88: 115, Resistor_SMD:R_0402_1005Metric
- removed R24, R59: 1.82k, Resistor_SMD:R_0402_1005Metric
- removed R25, R60: 100, Resistor_SMD:R_0402_1005Metric
- removed R3: 73.2k, Resistor_SMD:R_0402_1005Metric
- removed R32, R35: 16, Resistor_SMD:R_0402_1005Metric
- removed R41, R46: 19.1k, Resistor_SMD:R_0402_1005Metric
- removed R47, R53: 43k, Resistor_SMD:R_0402_1005Metric
- removed R48, R54: 27k, Resistor_SMD:R_0402_1005Metric
- removed R5: 3.9k, Resistor_SMD:R_0402_1005Metric
- removed R6: 1.3k, Resistor_SMD:R_0402_1005Metric
- removed R63, R65: 294, Resistor_SMD:R_0402_1005Metric
- removed R64: 17.8, Resistor_SMD:R_0402_1005Metric
- removed R66, R67, R68, R69: 47, Resistor_SMD:R_0402_1005Metric
- removed R7: 1M, Resistor_SMD:R_0603_1608Metric
- removed R71: 5.6k, Resistor_SMD:R_0402_1005Metric
- removed R89, R90, R91, R92: 51, Resistor_SMD:R_0402_1005Metric
- removed R95: 6.04k, Resistor_SMD:R_0402_1005Metric
- removed R96: 47k, Resistor_SMD:R_0402_1005Metric
- removed R97, R98: 100k, Resistor_SMD:R_0402_1005Metric
- removed R99: 5.24k, Resistor_SMD:R_0402_1005Metric
- removed SW1, SW10, SW12, SW13, SW14, SW16, SW17, SW18, SW2, SW20, SW21, SW22, SW3, SW4, SW5, SW6, SW8, SW9: SW_SPST, easyeda2kicad:KEY-SMD_L4.0-W3.0-LS4.9-1
- removed TP1, TP2, TP3, TP4: TestPoint, TestPoint:TestPoint_Pad_D1.5mm
- removed U1: ADR3425ARJZ-R7, easyeda2kicad:SOT-23-6_L2.9-W1.6-P0.95-LS2.8-BR
- removed U10, U17: PGA-103+, easyeda2kicad:SOT-89-3_L4.5-W2.4-P1.50-LS4.0-BR
- removed U11, U22, U29: PE4312C-Z, easyeda2kicad:QFN-20_L4.0-W4.0-P0.50-BL-EP2.2
- removed U12, U14, U36: ADF4351, Package_CSP:LFCSP-32-1EP_5x5mm_P0.5mm_EP3.25x3.25mm
- removed U13: ECS-TXO-2520MV-100-AY-TR, easyeda2kicad:OSC-SMD_4P-L2.5-W2.0-BL
- removed U15, U23: LT5560, Package_DFN_QFN:DFN-8-1EP_3x3mm_P0.5mm_EP1.66x2.38mm
- removed U16, U24: AD8342ACPZ-REEL7, easyeda2kicad:LFCSP-16_L3.0-W3.0-P0.50-TL-EP
- removed U18: ECS-TXO-2520-33-250-AN-TR, easyeda2kicad:OSC-SMD_4P-L2.5-W2.0-BL
- removed U19: OPA1612AxD, Package_SO:SOIC-8_3.9x4.9mm_P1.27mm
- removed U2: TPS564208DDCR, easyeda2kicad:SOT-23-6_L2.9-W1.6-P0.95-LS2.8-BR
- removed U20, U21: OPA354AIDBVR, easyeda2kicad:SOT-23-5_L3.0-W1.7-P0.95-LS2.8-BR
- removed U25: ADL5385ACPZ-R7, easyeda2kicad:LFCSP-24_L4.0-W4.0-P0.50-TL-EP2.3
- removed U26: ADA4940-2, Package_CSP:LFCSP-24-1EP_4x4mm_P0.5mm_EP2.5x2.5mm
- removed U27, U28, U31: PE4259-63, easyeda2kicad:SC-70-6_L2.2-W1.3-P0.65-LS2.1-BL
- removed U3: TPS563249DDCR, easyeda2kicad:TSOT-23-6_L2.9-W1.6-P0.95-LS2.8-TL
- removed U30: PSA4-5043+, easyeda2kicad:SOT-343-4_L2.0-W1.3-P1.30-LS2.1-BR
- removed U32, U33, U34, U35, U6, U7, U8, U9: BAR6402VH6327XTSA1, easyeda2kicad:SC-79_L1.2-W0.8-LS1.6-RD
- removed U38: BQ25798, Package_DFN_QFN:Texas_RQM0029A_VQFN-29_4x4mm_P0.4mm
- removed U39: MAX17205G_00E, lib:IC_MAX17205G_00E
- removed U4: LM2776, Package_TO_SOT_SMD:SOT-23-6
- removed U40: STM32H743VITx, Package_QFP:LQFP-100_14x14mm_P0.5mm
- removed U41: TLV320AIC3254IRHBT, easyeda2kicad:VQFN-32_L5.0-W5.0-P0.50-TL-EP
- removed U42: TPA2012D2RTJR, easyeda2kicad:QFN-20_L4.0-W4.0-P0.50-TL-EP2.7
- removed U43: RP2354A, Package_DFN_QFN:QFN-60-1EP_7x7mm_P0.4mm_EP3.4x3.4mm
- removed U44: ABM8-272-T3_C20625731, easyeda2kicad:CRYSTAL-SMD_4P-L3.2-W2.5-BL
- removed U45: MCP6002-xMC, Package_DFN_QFN:DFN-8-1EP_3x2mm_P0.5mm_EP1.75x1.45mm
- removed U5: LMV321, Package_TO_SOT_SMD:SOT-23-5
- removed USB1: TYPE-C 16PIN 2MD(073), easyeda2kicad:USB-C-SMD_TYPE-C-6PIN-2MD-073
- removed X1: XL2EL89COI-111YLC-25M, easyeda2kicad:CRYSTAL-SMD_4P-L3.2-W2.5-BL
- removed X2: Q13FC1350000400, easyeda2kicad:FC-135R_L3.2-W1.5
- removed Y1, Y3: ECS-96SMF45A30, lib:XTAL_ECS-96SMF45A30
- removed Y2: Si5351C-B-GM, Package_DFN_QFN:QFN-20-1EP_4x4mm_P0.5mm_EP2.7x2.7mm
