File: ht_better.kicad_sch (KiCad schematic)
At the start: 2 parts, among them J1 Conn_Coaxial

Commit message: add stuff
Other:
- added sheet Fuel Gauge (fuel_gauge.kicad_sch)
- added sheet MCU (mcu.kicad_sch)
- added sheet Peripherals (peripherals.kicad_sch)
- added sheet USB Type C (usb_c.kicad_sch)

Commit message: almost done with schematic
Other:
- removed sheet 2v5 Buffer
- added sheet RP2350 Slave (rp2350.kicad_sch)
- added sheet TX Bias Buffer (bias_buffer.kicad_sch)
- sheet MCU ports: added CHARGER_INT, CODEC_CS, CODEC_MISO, CODEC_MOSI, CODEC_NRST, CODEC_SCK, DISPLAY_CS, DISPLAY_ENABLE, DISPLAY_PWM, DISPLAY_RESET, DISPLAY_RS, DISPLAY_SCK, DISPLAY_SDA, FUNCTION_BTN, I2C_SCL, I2C_SDA, KEYPAD_COL1, KEYPAD_COL2, KEYPAD_COL3, KEYPAD_ROW1, KEYPAD_ROW2, KEYPAD_ROW3, KEYPAD_ROW4, KEYPAD_ROW5, PTT_BTN, PWR_SW, ROTARY_ENCODER_A, ROTARY_ENCODER_B, ROTARY_ENCODER_BTN, RP2350_CS, RP2350_MISO, RP2350_MOSI, RP2350_SCK, RX_IF_MIXER1_2M_EN, RX_IF_MIXER1_70CM_EN, RX_IF_MIXER2_2M_PWDN, RX_IF_MIXER2_70CM_PWDN, RX_IN_2M, RX_IN_70CM, SAI_BCLK, SAI_DIN, SAI_DOUT, SAI_MCLK, SAI_WCLK, SQUELCH_BTN, TR_SWITCH, TX_BAND_SWITCH1, TX_BAND_SWITCH2, TX_DRIVER_BIAS, TX_FDA_ENABLE, TX_FINALS_BIAS, TX_LPF_SWITCH1, TX_LPF_SWITCH2, TX_MIXER_ENABLE, USB_D+, USB_D-, VOL_POT; removed none
- sheet Peripherals ports: added CODEC_I2S_BCLK, CODEC_I2S_DIN, CODEC_I2S_DOUT, CODEC_I2S_MCLK, CODEC_I2S_WCLK, CODEC_NRST, CODEC_SPI_CS, CODEC_SPI_MISO, CODEC_SPI_MOSI, CODEC_SPI_SCLK, DISPLAY_CS, DISPLAY_ENABLE, DISPLAY_PWM, DISPLAY_RESET, DISPLAY_RS, DISPLAY_SCK, DISPLAY_SDA, FUNCTION_BUTTON, KEYPAD_COL1, KEYPAD_COL2, KEYPAD_COL3, KEYPAD_ROW1, KEYPAD_ROW2, KEYPAD_ROW3, KEYPAD_ROW4, KEYPAD_ROW5, OUT_HPL, OUT_HPR, POWER_SW, PTT_BUTTON, ROTARY_ENCODER_A, ROTARY_ENCODER_B, ROTARY_ENCODER_BTN, SQUELCH_BUTTON, VOLUME_POT; removed none
- sheet RF ports: added 1V25, TR_SWITCH; removed 2V5

Commit message: almost done assigning footprints
Parts:
- BT1: footprint (none) -> Connector_Wire:SolderWire-2.5sqmm_1x02_P7.2mm_D2.4mm_OD3.6mm
- J1: footprint (none) -> footprints:TE_CONSMA013.062
Changed lines of the file:
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@@
 			)
 		)
-		(property "Footprint" ""
+		(property "Footprint" "Connector_Wire:SolderWire-2.5sqmm_1x02_P7.2mm_D2.4mm_OD3.6mm"
 			(at 94.996 40.64 90)
 			(hide yes)
@@
 			)
 		)
-		(property "Footprint" ""
+		(property "Footprint" "footprints:TE_CONSMA013.062"
 			(at 36.83 53.34 0)
 			(hide yes)

Commit message: finish schematic
Parts:
- added R127, R128, R93, R94: 10k, symbol Device:R
Connections:
- net GND: now also R93.2, R94.2
- net MIXER1_2M_EN: now also R93.1
- net MIXER1_70CM_EN: now also R94.1
- net MIXER2_2M_PWDN: now also R127.1
- net MIXER2_70CM_PWDN: now also R128.1
- new net +3V3: R127.2, R128.2

Commit message: add connectors for b2b
Parts:
- added J4: ERF8-020-05.0-L-DV-L-K-TR, ERF8-020-05.0-L-DV-L-K-TR:SAMTEC_ERF8-020-05.0-L-DV-L-K-TR, symbol ERF8-020-05.0-L-DV-L-K-TR:ERF8-020-05.0-L-DV-L-K-TR
- added J5: ERM8-020-XX.X-X-DV-L-XX, ERM8-020-XX.X-X-DV-L-XX:SAMTEC_ERM8-020-XX.X-X-DV-L-XX, symbol ERM8-020-XX.X-X-DV-L-XX:ERM8-020-XX.X-X-DV-L-XX
- added R129, R130: 10k, symbol Device:R
Connections:
- net +3V3: now also J4.26, J4.28, J5.26, J5.28
- net 1V25: now also J4.30
- net GND: now also J4.01, J4.02, J4.05, J4.06, J4.09, J4.10, J4.14, J4.19, J4.20, J4.39, J5.01, J5.02, J5.05, J5.06, J5.09, J5.10, J5.14, J5.19, J5.20, J5.39, R129.2, R130.2
- net I2C_SCL: now also J4.16, J5.16
- net I2C_SDA: now also J4.18, J5.18
- net MIXER1_2M_EN: now also J4.33
- net MIXER1_70CM_EN: now also J4.35
- net MIXER2_2M_PWDN: now also J4.37
- net MIXER2_70CM_PWDN: now also J4.04
- net RP2350_CS: now also J4.11
- net RP2350_MISO: now also J4.13
- net RP2350_MOSI: now also J4.15
- net RP2350_SCK: now also J4.17
- net RX_2M: now also J4.08
- net RX_70CM: now also J4.12
- net TR_SWITCH: now also J4.21
- net TX_BAND_SWITCH1: now also J4.29
- net TX_BAND_SWITCH2: now also J4.31
- net TX_DRIVER_BIAS_BUF: now also J4.03
- net TX_FDA_DISABLE: now also R130.1
- net TX_FINAL_BIAS_BUF: now also J4.07
- net TX_LPF_SWITCH1: now also J4.23
- net TX_LPF_SWITCH2: now also J4.25
- net TX_MIXER_ENABLE: now also J4.27, R129.1
- new net +5V: J4.22, J4.24, J5.22, J5.24
- new net -5V: J4.32, J5.32
- new net 1V25_C: J5.30
- new net MIXER1_2M_EN_C: J5.33
- new net MIXER1_70CM_EN_C: J5.35
- new net MIXER2_2M_PWDN_C: J5.37
- new net MIXER2_70CM_PWDN_C: J5.04
- new net RP2350_CS_C: J5.11
- new net RP2350_MISO_C: J5.13
- new net RP2350_MOSI_C: J5.15
- new net RP2350_SCK_C: J5.17
- new net RX_2M_C: J5.08
- new net RX_70CM_C: J5.12
- new net TR_SWITCH_C: J5.21
- new net TX_BAND_SWITCH1_C: J5.29
- new net TX_BAND_SWITCH2_C: J5.31
- new net TX_DRIVER_BIAS_BUF_C: J5.03
- new net TX_FINAL_BIAS_BUF_C: J5.07
- new net TX_LPF_SWITCH1_C: J5.23
- new net TX_LPF_SWITCH2_C: J5.25
- new net TX_MIXER_ENABLE_C: J5.27
- new net VCC: J4.34, J4.36, J4.38, J4.40, J5.34, J5.36, J5.38, J5.40

Commit message: :3
Parts:
- J4: footprint ERF8-020-05.0-L-DV-L-K-TR:SAMTEC_ERF8-020-05.0-L-DV-L-K-TR -> footprints:SAMTEC_ERF8-020-05.0-L-DV-L-K-TR
- J5: footprint ERM8-020-XX.X-X-DV-L-XX:SAMTEC_ERM8-020-XX.X-X-DV-L-XX -> footprints:SAMTEC_ERM8-020-XX.X-X-DV-L-XX
- R127, R128, R129, R130, R93, R94: footprint (none) -> Resistor_SMD:R_0402_1005Metric
Changed lines of the file:
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@@
 			)
 		)
-		(property "Footprint" "ERF8-020-05.0-L-DV-L-K-TR:SAMTEC_ERF8-020-05.0-L-DV-L-K-TR"
+		(property "Footprint" "footprints:SAMTEC_ERF8-020-05.0-L-DV-L-K-TR"
 			(at 168.91 243.84 0)
 			(hide yes)
@@
 			)
 		)
-		(property "Footprint" ""
+		(property "Footprint" "Resistor_SMD:R_0402_1005Metric"
 			(at 59.69 254.762 90)
 			(hide yes)
@@
 			)
 		)
-		(property "Footprint" ""
+		(property "Footprint" "Resistor_SMD:R_0402_1005Metric"
 			(at 59.69 255.778 90)
 			(hide yes)
@@
 			)
 		)
-		(property "Footprint" ""
+		(property "Footprint" "Resistor_SMD:R_0402_1005Metric"
 			(at 59.69 236.728 90)
 			(hide yes)
@@
 			)
 		)
-		(property "Footprint" "ERM8-020-XX.X-X-DV-L-XX:SAMTEC_ERM8-020-XX.X-X-DV-L-XX"
+		(property "Footprint" "footprints:SAMTEC_ERM8-020-XX.X-X-DV-L-XX"
 			(at 236.22 243.84 0)
 			(hide yes)
@@
 			)
 		)
-		(property "Footprint" ""
+		(property "Footprint" "Resistor_SMD:R_0402_1005Metric"
 			(at 59.69 217.678 90)
 			(hide yes)
@@
 			)
 		)
-		(property "Footprint" ""
+		(property "Footprint" "Resistor_SMD:R_0402_1005Metric"
 			(at 59.69 235.712 90)
 			(hide yes)
@@
 			)
 		)
-		(property "Footprint" ""
+		(property "Footprint" "Resistor_SMD:R_0402_1005Metric"
 			(at 59.69 216.662 90)
 			(hide yes)
